Commit message: fmt & typos

File: aegis_description/urdf/adapter_from_sensor.xacro (robot description, xacro)
@@ -1,37 +1,36 @@
 <?xml version="1.0"?>
 <robot xmlns:xacro="http://ros.org/wiki/xacro">
-  <xacro:include filename="$(find aegis_description)/urdf/cylinders_inertial.xacro" />
+  <xacro:include filename="$(find aegis_description)/urdf/cylinders_inertial.xacro"/>
   <xacro:macro name="adapter_from_sensor" params="prefix parent">
-    <xacro:property name="mass" value="0.217" />
-    <xacro:property name="radius1" value="0.041" />
-    <xacro:property name="height1" value="0.0119" />
-    <xacro:property name="radius2" value="0.0315" />
-    <xacro:property name="height2" value="0.007" />
+    <xacro:property name="mass" value="0.217"/>
+    <xacro:property name="radius1" value="0.041"/>
+    <xacro:property name="height1" value="0.0119"/>
+    <xacro:property name="radius2" value="0.0315"/>
+    <xacro:property name="height2" value="0.007"/>
     <joint name="adapter_from_sensor_joint" type="fixed">
-      <origin xyz="0 0 ${height1}" rpy="0 0 0" />
-      <parent link="${parent}" />
-      <child link="${prefix}adapter_from_sensor" />
+      <origin xyz="0 0 ${height1}" rpy="0 0 0"/>
+      <parent link="${parent}"/>
+      <child link="${prefix}adapter_from_sensor"/>
     </joint>
     <link name="${prefix}adapter_from_sensor">
       <visual>
-        <origin xyz="0 0 0" rpy="0 0 0" />
+        <origin xyz="0 0 0" rpy="0 0 0"/>
         <geometry>
-          <mesh filename="package://aegis_description/meshes/adapter_from_sensor.dae"
-            scale="1.0 1.0 1.0" />
+          <mesh filename="package://aegis_description/meshes/adapter_from_sensor.dae" scale="1.0 1.0 1.0"/>
         </geometry>
       </visual>
-      <xacro:cylinders_inertial r1="${radius1}" l1="${height1}" r2="${radius2}" l2="${height2}" m="${mass}" />
+      <xacro:cylinders_inertial r1="${radius1}" l1="${height1}" r2="${radius2}" l2="${height2}" m="${mass}"/>
       <collision>
         <geometry>
-          <cylinder radius="${radius1}" length="${height1 + height2}" />
+          <cylinder radius="${radius1}" length="${height1 + height2}"/>
         </geometry>
       </collision>
     </link>
     <joint name="${prefix}adapter_from_sensor_end_joint" type="fixed">
-      <origin xyz="0 0 ${height2}" rpy="0 0 0" />
-      <parent link="${prefix}adapter_from_sensor" />
-      <child link="${prefix}adapter_from_sensor_end" />
+      <origin xyz="0 0 ${height2}" rpy="0 0 0"/>
+      <parent link="${prefix}adapter_from_sensor"/>
+      <child link="${prefix}adapter_from_sensor_end"/>
     </joint>
-    <link name="${prefix}adapter_from_sensor_end" />
+    <link name="${prefix}adapter_from_sensor_end"/>
   </xacro:macro>
 </robot>

File: aegis_description/urdf/adapter_to_sensor.xacro (robot description, xacro)
@@ -1,50 +1,49 @@
 <?xml version="1.0"?>
 <robot xmlns:xacro="http://ros.org/wiki/xacro">
-  <xacro:include filename="$(find aegis_description)/urdf/cylinders_inertial.xacro" />
+  <xacro:include filename="$(find aegis_description)/urdf/cylinders_inertial.xacro"/>
   <xacro:macro name="adapter_to_sensor" params="prefix parent">
-    <xacro:property name="mass" value="0.242" />
-    <xacro:property name="radius1" value="0.03025" />
-    <xacro:property name="height1" value="0.0116" />
-    <xacro:property name="radius2" value="0.04255" />
-    <xacro:property name="height2" value="0.0094" />
+    <xacro:property name="mass" value="0.242"/>
+    <xacro:property name="radius1" value="0.03025"/>
+    <xacro:property name="height1" value="0.0116"/>
+    <xacro:property name="radius2" value="0.04255"/>
+    <xacro:property name="height2" value="0.0094"/>
     <joint name="${prefix}adapter_to_sensor_joint" type="fixed">
-      <origin xyz="0 0 0" rpy="0 0 0" />
-      <parent link="${parent}" />
-      <child link="${prefix}adapter_to_sensor" />
+      <origin xyz="0 0 0" rpy="0 0 0"/>
+      <parent link="${parent}"/>
+      <child link="${prefix}adapter_to_sensor"/>
     </joint>
     <link name="${prefix}adapter_to_sensor">
       <visual>
-        <origin xyz="0 0 ${0.5 * height1}" rpy="0 0 0" />
+        <origin xyz="0 0 ${0.5 * height1}" rpy="0 0 0"/>
         <geometry>
-          <cylinder radius="${radius1}" length="${height1}" />
+          <cylinder radius="${radius1}" length="${height1}"/>
         </geometry>
         <material name="black">
-          <color rgba="0.04 0.04 0.04 1" />
+          <color rgba="0.04 0.04 0.04 1"/>
         </material>
       </visual>
       <visual>
-        <origin xyz="0 0 ${height1 + 0.5 * height2}" rpy="0 0 0" />
+        <origin xyz="0 0 ${height1 + 0.5 * height2}" rpy="0 0 0"/>
         <geometry>
-          <cylinder radius="${radius2}" length="${height2}" />
+          <cylinder radius="${radius2}" length="${height2}"/>
         </geometry>
         <material name="black">
-          <color rgba="0.04 0.04 0.04 1" />
+          <color rgba="0.04 0.04 0.04 1"/>
         </material>
       </visual>
-      <xacro:cylinders_inertial r1="${radius1}" l1="${height1}" r2="${radius2}" l2="${height2}"
-        m="${mass}" />
+      <xacro:cylinders_inertial r1="${radius1}" l1="${height1}" r2="${radius2}" l2="${height2}" m="${mass}"/>
       <collision>
-        <origin xyz="0 0 ${0.5 * (height1 + height2)}" rpy="0 0 0" />
+        <origin xyz="0 0 ${0.5 * (height1 + height2)}" rpy="0 0 0"/>
         <geometry>
-          <cylinder radius="${radius2}" length="${height1 + height2}" />
+          <cylinder radius="${radius2}" length="${height1 + height2}"/>
         </geometry>
       </collision>
     </link>
     <joint name="${prefix}adapter_to_sensor_end_joint" type="fixed">
-      <origin xyz="0 0 ${height1 + height2}" rpy="0 0 0" />
-      <parent link="${prefix}adapter_to_sensor" />
-      <child link="${prefix}adapter_to_sensor_end" />
+      <origin xyz="0 0 ${height1 + height2}" rpy="0 0 0"/>
+      <parent link="${prefix}adapter_to_sensor"/>
+      <child link="${prefix}adapter_to_sensor_end"/>
     </joint>
-    <link name="${prefix}adapter_to_sensor_end" />
+    <link name="${prefix}adapter_to_sensor_end"/>
   </xacro:macro>
 </robot>

File: aegis_description/urdf/aegis.urdf.xacro (robot description, xacro)
@@ -1,16 +1,16 @@
 <?xml version="1.0"?>
 <robot xmlns:xacro="http://wiki.ros.org/xacro" name="aegis">
-  <xacro:arg name="name" default="aegis" />
-  <xacro:arg name="kinematics_params" default="$(find ur_description)/config/ur5e/default_kinematics.yaml" />
-  <xacro:include filename="$(find aegis_description)/urdf/ur_definition.xacro" />
-  <xacro:include filename="$(find aegis_description)/urdf/adapter_to_sensor.xacro" />
-  <xacro:include filename="$(find aegis_description)/urdf/ft_schunk_axia80.xacro" />
-  <xacro:include filename="$(find aegis_description)/urdf/adapter_from_sensor.xacro" />
-  <xacro:include filename="$(find robotiq_hande_description)/urdf/robotiq_hande_gripper.xacro" />
-  <link name="ur_base" />
-  <xacro:ur_definition name="$(arg name)" kinematics_params="$(arg kinematics_params)" />
-  <xacro:adapter_to_sensor parent="tool0" prefix="" />
-  <xacro:ft_sensor_schunk_axia80 parent="adapter_to_sensor_end" prefix="" />
-  <xacro:adapter_from_sensor parent="tool_mount_link" prefix="" />
-  <xacro:robotiq_hande_gripper parent="adapter_from_sensor_end" prefix="" />
+  <xacro:arg name="name" default="aegis"/>
+  <xacro:arg name="kinematics_params" default="$(find ur_description)/config/ur5e/default_kinematics.yaml"/>
+  <xacro:include filename="$(find aegis_description)/urdf/ur_definition.xacro"/>
+  <xacro:include filename="$(find aegis_description)/urdf/adapter_to_sensor.xacro"/>
+  <xacro:include filename="$(find aegis_description)/urdf/ft_schunk_axia80.xacro"/>
+  <xacro:include filename="$(find aegis_description)/urdf/adapter_from_sensor.xacro"/>
+  <xacro:include filename="$(find robotiq_hande_description)/urdf/robotiq_hande_gripper.xacro"/>
+  <link name="ur_base"/>
+  <xacro:ur_definition name="$(arg name)" kinematics_params="$(arg kinematics_params)"/>
+  <xacro:adapter_to_sensor parent="tool0" prefix=""/>
+  <xacro:ft_sensor_schunk_axia80 parent="adapter_to_sensor_end" prefix=""/>
+  <xacro:adapter_from_sensor parent="tool_mount_link" prefix=""/>
+  <xacro:robotiq_hande_gripper parent="adapter_from_sensor_end" prefix=""/>
 </robot>

File: aegis_description/urdf/cylinders_inertial.xacro (robot description, xacro)
@@ -3,5 +3,5 @@
   <xacro:macro name="cylinders_inertial" params="r1 l1 r2 l2 m">
     <inertial>
-      <mass value="${m}" />
+      <mass value="${m}"/>
       <inertia
         ixx="${0.0833333 * m * (3 * (r1 * r1 + r2 * r2) + l1 * l1 + l2 * l2)}"
@@ -10,5 +10,6 @@
         iyy="${0.0833333 * m * (3 * (r1 * r1 + r2 * r2) + l1 * l1 + l2 * l2)}"
         iyz="0.0"
-        izz="${0.5 * m * (r1 * r1 + r2 * r2)}" />
+        izz="${0.5 * m * (r1 * r1 + r2 * r2)}"
+      />
     </inertial>
   </xacro:macro>

File: aegis_description/urdf/ft_schunk_axia80.xacro (robot description, xacro)
@@ -1,28 +1,29 @@
 <?xml version="1.0"?>
 <robot xmlns:xacro="http://ros.org/wiki/xacro">
-    <!--
+  <!--
         SCHUNK AXIA80 F/T Sensor
     -->
-    <xacro:arg name="use_physical_hardware" default="false" />
-    <xacro:arg name="ip_address" default="127.0.0.1" />
-    <xacro:arg name="rdt_sampling_rate" default="500" />
-    <xacro:arg name="sensor_type" default="ati_axia80" />
-    <xacro:arg name="bolts_mass" default="0.019" />
-    <xacro:arg name="internal_filter_rate" default="0" />
-    <xacro:arg name="use_hardware_biasing" default="false" />
-    <xacro:include filename="$(find net_ft_description)/urdf/net_ft_sensor.xacro" />
-    <xacro:macro name="ft_sensor_schunk_axia80" params="prefix parent">
-        <xacro:net_ft_sensor
-            parent="${parent}"
-            prefix="${prefix}"
-            use_physical_hardware="$(arg use_physical_hardware)"
-            ip_address="$(arg ip_address)"
-            rdt_sampling_rate="$(arg rdt_sampling_rate)"
-            sensor_type="$(arg sensor_type)"
-            bolts_mass="$(arg bolts_mass)"
-            internal_filter_rate="$(arg internal_filter_rate)"
-            use_hardware_biasing="$(arg use_hardware_biasing)">
-            <origin xyz="0 0 0" rpy="0 0 0" />
-        </xacro:net_ft_sensor>
-    </xacro:macro>
+  <xacro:arg name="use_physical_hardware" default="false"/>
+  <xacro:arg name="ip_address" default="127.0.0.1"/>
+  <xacro:arg name="rdt_sampling_rate" default="500"/>
+  <xacro:arg name="sensor_type" default="ati_axia80"/>
+  <xacro:arg name="bolts_mass" default="0.019"/>
+  <xacro:arg name="internal_filter_rate" default="0"/>
+  <xacro:arg name="use_hardware_biasing" default="false"/>
+  <xacro:include filename="$(find net_ft_description)/urdf/net_ft_sensor.xacro"/>
+  <xacro:macro name="ft_sensor_schunk_axia80" params="prefix parent">
+    <xacro:net_ft_sensor
+      parent="${parent}"
+      prefix="${prefix}"
+      use_physical_hardware="$(arg use_physical_hardware)"
+      ip_address="$(arg ip_address)"
+      rdt_sampling_rate="$(arg rdt_sampling_rate)"
+      sensor_type="$(arg sensor_type)"
+      bolts_mass="$(arg bolts_mass)"
+      internal_filter_rate="$(arg internal_filter_rate)"
+      use_hardware_biasing="$(arg use_hardware_biasing)"
+    >
+      <origin xyz="0 0 0" rpy="0 0 0"/>
+    </xacro:net_ft_sensor>
+  </xacro:macro>
 </robot>
