Commit message: Integrate cell into Aegis Xacro model

File: aegis_description/urdf/aegis.urdf.xacro (robot description, xacro)
@@ -3,4 +3,5 @@
   <xacro:arg name="name" default="aegis"/>
   <xacro:arg name="kinematics_params" default="$(find ur_description)/config/ur5e/default_kinematics.yaml"/>
+  <xacro:include filename="$(find aegis_description)/urdf/cell.xacro"/>
   <xacro:include filename="$(find aegis_description)/urdf/ur_definition.xacro"/>
   <xacro:include filename="$(find aegis_description)/urdf/adapter_to_sensor.xacro"/>
@@ -8,5 +9,6 @@
   <xacro:include filename="$(find aegis_description)/urdf/adapter_from_sensor.xacro"/>
   <xacro:include filename="$(find robotiq_hande_description)/urdf/robotiq_hande_gripper.xacro"/>
-  <link name="ur_base"/>
+  <link name="world" />
+  <xacro:cell parent="world" />
   <xacro:ur_definition name="$(arg name)" kinematics_params="$(arg kinematics_params)"/>
   <xacro:adapter_to_sensor parent="tool0" prefix=""/>

Commit message: Format

File: aegis_description/urdf/aegis.urdf.xacro (robot description, xacro)
@@ -9,6 +9,6 @@
   <xacro:include filename="$(find aegis_description)/urdf/adapter_from_sensor.xacro"/>
   <xacro:include filename="$(find robotiq_hande_description)/urdf/robotiq_hande_gripper.xacro"/>
-  <link name="world" />
-  <xacro:cell parent="world" />
+  <link name="world"/>
+  <xacro:cell parent="world"/>
   <xacro:ur_definition name="$(arg name)" kinematics_params="$(arg kinematics_params)"/>
   <xacro:adapter_to_sensor parent="tool0" prefix=""/>

File: aegis_description/urdf/cell.xacro (robot description, xacro)
@@ -3,30 +3,28 @@
   <xacro:macro name="cell" params="parent">
     <joint name="world_to_cell_joint" type="fixed">
-      <origin xyz="0 0 0" rpy="0 0 0" />
-      <parent link="${parent}" />
-      <child link="cell" />
+      <origin xyz="0 0 0" rpy="0 0 0"/>
+      <parent link="${parent}"/>
+      <child link="cell"/>
     </joint>
     <link name="cell">
       <visual>
-        <origin xyz="-0.460 -0.240 0.786" rpy="0 0 0" />
+        <origin xyz="-0.460 -0.240 0.786" rpy="0 0 0"/>
         <geometry>
-          <mesh filename="package://aegis_description/meshes/cell.dae"
-            scale="1.0 1.0 1.0" />
+          <mesh filename="package://aegis_description/meshes/cell.dae" scale="1.0 1.0 1.0"/>
         </geometry>
       </visual>
       <collision>
-        <origin xyz="-0.460 -0.240 0.786" rpy="0 0 0" />
+        <origin xyz="-0.460 -0.240 0.786" rpy="0 0 0"/>
         <geometry>
-          <mesh filename="package://aegis_description/meshes/cell.dae"
-            scale="1.0 1.0 1.0" />
+          <mesh filename="package://aegis_description/meshes/cell.dae" scale="1.0 1.0 1.0"/>
         </geometry>
       </collision>
     </link>
     <joint name="cell_to_ur_base" type="fixed">
-      <origin xyz="0 0 0.806" rpy="0 0 ${0.5 * pi}" />
-      <parent link="cell" />
-      <child link="ur_base" />
+      <origin xyz="0 0 0.806" rpy="0 0 ${0.5 * pi}"/>
+      <parent link="cell"/>
+      <child link="ur_base"/>
     </joint>
-    <link name="ur_base" />
+    <link name="ur_base"/>
   </xacro:macro>
 </robot>

Commit message: moved & renamed files

File: aegis_description/urdf/aegis.urdf.xacro (robot description, xacro)
@@ -2,15 +2,6 @@
 <robot xmlns:xacro="http://wiki.ros.org/xacro" name="aegis">
   <xacro:arg name="name" default="aegis"/>
-  <xacro:arg name="kinematics_params" default="$(find ur_description)/config/ur5e/default_kinematics.yaml"/>
-  <xacro:include filename="$(find aegis_description)/urdf/ur_definition.xacro"/>
-  <xacro:include filename="$(find aegis_description)/urdf/adapter_to_sensor.xacro"/>
-  <xacro:include filename="$(find aegis_description)/urdf/ft_schunk_axia80.xacro"/>
-  <xacro:include filename="$(find aegis_description)/urdf/adapter_from_sensor.xacro"/>
-  <xacro:include filename="$(find robotiq_hande_description)/urdf/robotiq_hande_gripper.xacro"/>
+  <xacro:include filename="$(find aegis_description)/urdf/aegis.xacro"/>
   <link name="ur_base"/>
-  <xacro:ur_definition name="$(arg name)" kinematics_params="$(arg kinematics_params)"/>
-  <xacro:adapter_to_sensor parent="tool0" prefix=""/>
-  <xacro:ft_sensor_schunk_axia80 parent="adapter_to_sensor_end" prefix=""/>
-  <xacro:adapter_from_sensor parent="tool_mount_link" prefix=""/>
-  <xacro:robotiq_hande_gripper parent="adapter_from_sensor_end" prefix=""/>
+  <xacro:aegis_robot name="$(arg name)" parent="ur_base" prefix=""/>
 </robot>

File: aegis_description/urdf/modules/ft_schunk_axia80.xacro (robot description, xacro)
@@ -12,5 +12,6 @@
   <xacro:arg name="use_hardware_biasing" default="false"/>
   <xacro:include filename="$(find net_ft_description)/urdf/net_ft_sensor.xacro"/>
-  <xacro:macro name="ft_sensor_schunk_axia80" params="prefix parent">
+  <xacro:macro name="ft_sensor_schunk_axia80" params="prefix parent fake_hardware">
+    <!-- TODO: include the fake_hardware param -->
     <xacro:net_ft_sensor
       parent="${parent}"

File: aegis_description/urdf/modules/ur_definition.xacro (robot description, xacro)
@@ -2,5 +2,5 @@
 <robot xmlns:xacro="http://ros.org/wiki/xacro">
   <xacro:include filename="$(find ur_description)/urdf/ur_macro.xacro"/>
-  <xacro:macro name="ur_definition" params="name kinematics_params">
+  <xacro:macro name="ur_definition" params="name kinematics_params fake_hardware">
     <!-- possible 'ur_type' values: ur3, ur3e, ur5, ur5e, ur10, ur10e, ur16e, ur20 -->
     <!-- the default value should raise an error in case this was called without defining the
@@ -39,10 +39,11 @@
     <xacro:arg name="tool_tcp_port" default="54321"/>
     <!-- Simulation parameters -->
-    <xacro:arg name="use_fake_hardware" default="true"/>
-    <xacro:arg name="fake_sensor_commands" default="false"/>
+    <xacro:arg name="use_fake_hardware" default="$(arg fake_hardware)"/>
+    <xacro:arg name="fake_sensor_commands" default="$(arg fake_hardware)"/>
     <xacro:arg name="sim_gazebo" default="false"/>
     <xacro:arg name="sim_ignition" default="false"/>
     <xacro:arg name="simulation_controllers" default=""/>
     <!-- initial position for simulations (Fake Hardware, Gazebo, Ignition) -->
+    <!-- TODO: remap this to our aegis_control package -->
     <xacro:arg name="initial_positions_file" default="$(find ur_description)/config/initial_positions.yaml"/>
     <!-- convert to property to use substitution in function -->

Commit message: moved & renamed files

File: aegis_description/urdf/aegis.urdf.xacro (robot description, xacro)
@@ -1,7 +1,13 @@
 <?xml version="1.0"?>
 <robot xmlns:xacro="http://wiki.ros.org/xacro" name="aegis">
-  <xacro:arg name="name" default="aegis"/>
+  <xacro:arg name="mock_hardware" default="false"/>
+  <xacro:arg name="base_link" default="ur_base"/>
+  <xacro:arg name="prefix" default=""/>
+  <xacro:arg name="initial_positions_file" default="$(find aegis_description)/config/initial_positions.yaml"/>
   <xacro:include filename="$(find aegis_description)/urdf/aegis.xacro"/>
-  <link name="ur_base"/>
-  <xacro:aegis_robot name="$(arg name)" parent="ur_base" prefix=""/>
+  <xacro:include filename="$(find aegis_description)/urdf/aegis.control.xacro"/>
+  <link name="$(arg base_link)"/>
+  <xacro:aegis_robot parent="$(arg base_link)" prefix="$(arg prefix)" mock_hardware="$(arg mock_hardware)"/>
+  <!-- TODO: VERIFY IF CUSTOM ROS2 CONTROL FILE IS NEEDED FOR OUR SETUP SINCE UR_ROBOT_DRIVER DOES SOMETHING -->
+  <xacro:aegis_ros2_control initial_positions_file="$(arg initial_positions_file)" mock_hardware="$(arg mock_hardware)"/>
 </robot>

File: aegis_description/urdf/modules/ur_definition.xacro (robot description, xacro)
@@ -4,5 +4,5 @@
   <!-- The list of all available options can be found in the <ur_description>/ur_macro.xacro file -->
   <!-- Descriptions of the arguments can be found in the <ur_robot_driver>/src/hardware_interface.cpp file -->
-  <xacro:macro name="ur_definition" params="name parent prefix kinematics_calibration mock_hardware">
+  <xacro:macro name="ur_definition" params="name parent prefix mock_hardware">
     <!-- parameters -->
     <xacro:arg name="tf_prefix" default="${prefix}"/>
@@ -31,4 +31,5 @@
     <!-- initial position for simulations (Fake Hardware, Gazebo, Ignition) -->
     <xacro:arg name="initial_positions_file" default="$(find aegis_control)/config/initial_positions.yaml"/>
+    <xacro:arg name="kinematics_calibration" default="$(find aegis_description)/config/ur5e/calibration.yaml"/>
     <!-- convert to property to use substitution in function -->
     <xacro:property name="initial_positions_file" default="$(arg initial_positions_file)"/>
@@ -39,5 +40,5 @@
       parent="${parent}"
       joint_limits_parameters_file="$(arg joint_limit_params)"
-      kinematics_parameters_file="${kinematics_calibration}"
+      kinematics_parameters_file="$(arg kinematics_calibration)"
       physical_parameters_file="$(arg physical_params)"
       visual_parameters_file="$(arg visual_params)"

Commit message: added tf_prefix to the bringup file

File: aegis_description/urdf/aegis.urdf.xacro (robot description, xacro)
@@ -4,7 +4,8 @@
   <xacro:arg name="base_link" default="ur_base"/>
   <xacro:arg name="prefix" default=""/>
+  <xacro:arg name="tf_prefix" default=""/>
   <xacro:arg name="initial_positions_file" default="$(find aegis_description)/config/initial_positions.yaml"/>
   <xacro:include filename="$(find aegis_description)/urdf/aegis.xacro"/>
   <link name="$(arg base_link)"/>
-  <xacro:aegis_robot parent="$(arg base_link)" prefix="$(arg prefix)" mock_hardware="$(arg mock_hardware)"/>
+  <xacro:aegis_robot parent="$(arg base_link)" tf_prefix="$(arg tf_prefix)" prefix="$(arg prefix)" mock_hardware="$(arg mock_hardware)"/>
 </robot>

File: aegis_description/urdf/aegis.xacro (robot description, xacro)
@@ -6,6 +6,6 @@
   <xacro:include filename="$(find aegis_description)/urdf/modules/adapter_from_sensor.xacro"/>
   <xacro:include filename="$(find robotiq_hande_description)/urdf/robotiq_hande_gripper.xacro"/>
-  <xacro:macro name="aegis_robot" params="parent prefix mock_hardware">
-    <xacro:ur_definition name="aegis" parent="${parent}" prefix="${prefix}" mock_hardware="${mock_hardware}"/>
+  <xacro:macro name="aegis_robot" params="parent tf_prefix prefix mock_hardware">
+    <xacro:ur_definition name="aegis" parent="${parent}" tf_prefix="${tf_prefix}" mock_hardware="${mock_hardware}"/>
     <xacro:adapter_to_sensor parent="tool0" prefix="${prefix}"/>
     <xacro:ft_sensor_schunk_axia80 parent="adapter_to_sensor_end" prefix="${prefix}" mock_hardware="${mock_hardware}"/>

File: aegis_description/urdf/modules/ur_definition.xacro (robot description, xacro)
@@ -4,7 +4,7 @@
   <!-- The list of all available options can be found in the <ur_description>/ur_macro.xacro file -->
   <!-- Descriptions of the arguments can be found in the <ur_robot_driver>/src/hardware_interface.cpp file -->
-  <xacro:macro name="ur_definition" params="name parent prefix mock_hardware">
+  <xacro:macro name="ur_definition" params="name parent tf_prefix mock_hardware">
     <!-- parameters -->
-    <xacro:arg name="tf_prefix" default="${prefix}"/>
+    <xacro:arg name="tf_prefix" default="${tf_prefix}"/>
     <xacro:arg name="joint_limit_params" default="$(find aegis_description)/config/ur5e/joint_limits.yaml"/>
     <xacro:arg name="physical_params" default="$(find aegis_description)/config/ur5e/physical_parameters.yaml"/>

Commit message: Add robot cell (#8)

File: aegis_description/urdf/aegis.urdf.xacro (robot description, xacro)
@@ -3,4 +3,6 @@
   <xacro:arg name="name" default="aegis"/>
   <xacro:arg name="kinematics_params" default="$(find ur_description)/config/ur5e/default_kinematics.yaml"/>
+  <xacro:include filename="$(find aegis_description)/urdf/cell.xacro"/>
+  <xacro:include filename="$(find aegis_description)/urdf/oakd_pro_camera.xacro"/>
   <xacro:include filename="$(find aegis_description)/urdf/ur_definition.xacro"/>
   <xacro:include filename="$(find aegis_description)/urdf/adapter_to_sensor.xacro"/>
@@ -8,5 +10,7 @@
   <xacro:include filename="$(find aegis_description)/urdf/adapter_from_sensor.xacro"/>
   <xacro:include filename="$(find robotiq_hande_description)/urdf/robotiq_hande_gripper.xacro"/>
-  <link name="ur_base"/>
+  <link name="world"/>
+  <xacro:cell parent="world"/>
+  <xacro:oakd_pro_camera parent="cell"/>
   <xacro:ur_definition name="$(arg name)" kinematics_params="$(arg kinematics_params)"/>
   <xacro:adapter_to_sensor parent="tool0" prefix=""/>

Commit message: LaunchFiles totaly makeover - `mock_hardware` & `launch_rviz` params (#9)

File: aegis_description/urdf/aegis.urdf.xacro (robot description, xacro)
@@ -1,20 +1,10 @@
 <?xml version="1.0"?>
 <robot xmlns:xacro="http://wiki.ros.org/xacro" name="aegis">
-  <xacro:arg name="name" default="aegis"/>
-  <xacro:arg name="kinematics_params" default="$(find ur_description)/config/ur5e/default_kinematics.yaml"/>
-  <xacro:include filename="$(find aegis_description)/urdf/cell.xacro"/>
-  <xacro:include filename="$(find aegis_description)/urdf/oakd_pro_camera.xacro"/>
-  <xacro:include filename="$(find aegis_description)/urdf/ur_definition.xacro"/>
-  <xacro:include filename="$(find aegis_description)/urdf/adapter_to_sensor.xacro"/>
-  <xacro:include filename="$(find aegis_description)/urdf/ft_schunk_axia80.xacro"/>
-  <xacro:include filename="$(find aegis_description)/urdf/adapter_from_sensor.xacro"/>
-  <xacro:include filename="$(find robotiq_hande_description)/urdf/robotiq_hande_gripper.xacro"/>
-  <link name="world"/>
-  <xacro:cell parent="world"/>
-  <xacro:oakd_pro_camera parent="cell"/>
-  <xacro:ur_definition name="$(arg name)" kinematics_params="$(arg kinematics_params)"/>
-  <xacro:adapter_to_sensor parent="tool0" prefix=""/>
-  <xacro:ft_sensor_schunk_axia80 parent="adapter_to_sensor_end" prefix=""/>
-  <xacro:adapter_from_sensor parent="tool_mount_link" prefix=""/>
-  <xacro:robotiq_hande_gripper parent="adapter_from_sensor_end" prefix=""/>
+  <xacro:arg name="mock_hardware" default="false"/>
+  <xacro:arg name="base_link" default="world"/>
+  <xacro:arg name="prefix" default=""/>
+  <xacro:arg name="tf_prefix" default=""/>
+  <xacro:include filename="$(find aegis_description)/urdf/aegis.xacro"/>
+  <link name="$(arg base_link)"/>
+  <xacro:aegis_robot parent="$(arg base_link)" tf_prefix="$(arg tf_prefix)" prefix="$(arg prefix)" mock_hardware="$(arg mock_hardware)"/>
 </robot>

File: aegis_description/urdf/modules/ft_schunk_axia80.xacro (robot description, xacro)
@@ -12,9 +12,9 @@
   <xacro:arg name="use_hardware_biasing" default="false"/>
   <xacro:include filename="$(find net_ft_description)/urdf/net_ft_sensor.xacro"/>
-  <xacro:macro name="ft_sensor_schunk_axia80" params="prefix parent">
+  <xacro:macro name="ft_sensor_schunk_axia80" params="prefix parent mock_hardware">
     <xacro:net_ft_sensor
       parent="${parent}"
       prefix="${prefix}"
-      use_physical_hardware="$(arg use_physical_hardware)"
+      use_physical_hardware="${mock_hardware == 'false'}"
       ip_address="$(arg ip_address)"
       rdt_sampling_rate="$(arg rdt_sampling_rate)"

File: aegis_description/urdf/modules/ur_definition.xacro (robot description, xacro)
@@ -2,60 +2,47 @@
 <robot xmlns:xacro="http://ros.org/wiki/xacro">
   <xacro:include filename="$(find ur_description)/urdf/ur_macro.xacro"/>
-  <xacro:macro name="ur_definition" params="name kinematics_params">
-    <!-- possible 'ur_type' values: ur3, ur3e, ur5, ur5e, ur10, ur10e, ur16e, ur20 -->
-    <!-- the default value should raise an error in case this was called without defining the
-        type -->
-    <xacro:arg name="ur_type" default="ur5e"/>
+  <!-- The list of all available options can be found in the <ur_description>/urdf/ur_macro.xacro file -->
+  <!-- Descriptions of the arguments can be found in the <ur_robot_driver>/src/hardware_interface.cpp file -->
+  <xacro:macro name="ur_definition" params="name parent tf_prefix mock_hardware">
     <!-- parameters -->
-    <xacro:arg name="tf_prefix" default=""/>
-    <!-- TODO(issue#1): It must be updated with real hardware paramas! -->
-    <xacro:arg name="joint_limit_params" default="$(find ur_description)/config/$(arg ur_type)/joint_limits.yaml"/>
-    <xacro:arg name="physical_params" default="$(find ur_description)/config/$(arg ur_type)/physical_parameters.yaml"/>
-    <xacro:arg name="visual_params" default="$(find ur_description)/config/$(arg ur_type)/visual_parameters.yaml"/>
-    <xacro:arg name="transmission_hw_interface" default=""/>
+    <xacro:arg name="tf_prefix" default="${tf_prefix}"/>
+    <xacro:arg name="joint_limit_params" default="$(find aegis_description)/config/ur5e/joint_limits.yaml"/>
+    <xacro:arg name="physical_params" default="$(find aegis_description)/config/ur5e/physical_parameters.yaml"/>
+    <xacro:arg name="visual_params" default="$(find aegis_description)/config/ur5e/visual_parameters.yaml"/>
+    <!-- ros2_control side safety -->
     <xacro:arg name="safety_limits" default="true"/>
     <xacro:arg name="safety_pos_margin" default="0.15"/>
     <xacro:arg name="safety_k_position" default="20"/>
     <!-- ros2_control related parameters -->
-    <xacro:arg name="headless_mode" default="false"/>
-    <xacro:arg name="robot_ip" default="0.0.0.0"/>
-    <xacro:arg name="script_filename" default=""/>
+    <xacro:arg name="robot_ip" default="aegis_ur"/>
+    <xacro:arg name="script_filename" default="$(find ur_robot_driver)/resources/ros_control.urscript"/>
     <xacro:arg name="output_recipe_filename" default="$(find ur_robot_driver)/resources/rtde_output_recipe.txt"/>
     <xacro:arg name="input_recipe_filename" default="$(find ur_robot_driver)/resources/rtde_input_recipe.txt"/>
     <xacro:arg name="reverse_ip" default="0.0.0.0"/>
-    <xacro:arg name="script_command_port" default="50004"/>
-    <xacro:arg name="reverse_port" default="50001"/>
-    <xacro:arg name="script_sender_port" default="50002"/>
-    <xacro:arg name="trajectory_port" default="50003"/>
     <!--   tool communication related parameters-->
     <xacro:arg name="use_tool_communication" default="false"/>
     <xacro:arg name="tool_voltage" default="0"/>
-    <xacro:arg name="tool_parity" default="0"/>
-    <xacro:arg name="tool_baud_rate" default="115200"/>
-    <xacro:arg name="tool_stop_bits" default="1"/>
-    <xacro:arg name="tool_rx_idle_chars" default="1.5"/>
-    <xacro:arg name="tool_tx_idle_chars" default="3.5"/>
     <xacro:arg name="tool_device_name" default="/tmp/ttyUR"/>
-    <xacro:arg name="tool_tcp_port" default="54321"/>
     <!-- Simulation parameters -->
-    <xacro:arg name="use_fake_hardware" default="true"/>
-    <xacro:arg name="fake_sensor_commands" default="false"/>
+    <xacro:arg name="use_fake_hardware" default="${str(mock_hardware)}"/>
+    <xacro:arg name="fake_sensor_commands" default="${str(mock_hardware)}"/>
+    <xacro:arg name="headless_mode" default="false"/>
     <xacro:arg name="sim_gazebo" default="false"/>
     <xacro:arg name="sim_ignition" default="false"/>
     <xacro:arg name="simulation_controllers" default=""/>
     <!-- initial position for simulations (Fake Hardware, Gazebo, Ignition) -->
-    <xacro:arg name="initial_positions_file" default="$(find ur_description)/config/initial_positions.yaml"/>
+    <xacro:arg name="initial_positions_file" default="$(find aegis_description)/config/initial_positions.yaml"/>
+    <xacro:arg name="kinematics_calibration" default="$(find aegis_description)/config/ur5e/calibration.yaml"/>
     <!-- convert to property to use substitution in function -->
     <xacro:property name="initial_positions_file" default="$(arg initial_positions_file)"/>
     <!-- arm -->
     <xacro:ur_robot
-      name="aegis"
+      name="${name}"
       tf_prefix="$(arg tf_prefix)"
-      parent="ur_base"
+      parent="${parent}"
       joint_limits_parameters_file="$(arg joint_limit_params)"
-      kinematics_parameters_file="$(arg kinematics_params)"
+      kinematics_parameters_file="$(arg kinematics_calibration)"
       physical_parameters_file="$(arg physical_params)"
       visual_parameters_file="$(arg visual_params)"
-      transmission_hw_interface="$(arg transmission_hw_interface)"
       safety_limits="$(arg safety_limits)"
       safety_pos_margin="$(arg safety_pos_margin)"
@@ -63,17 +50,11 @@
       use_fake_hardware="$(arg use_fake_hardware)"
       fake_sensor_commands="$(arg fake_sensor_commands)"
+      headless_mode="$(arg headless_mode)"
       sim_gazebo="$(arg sim_gazebo)"
       sim_ignition="$(arg sim_ignition)"
-      headless_mode="$(arg headless_mode)"
       initial_positions="${xacro.load_yaml(initial_positions_file)}"
       use_tool_communication="$(arg use_tool_communication)"
       tool_voltage="$(arg tool_voltage)"
-      tool_parity="$(arg tool_parity)"
-      tool_baud_rate="$(arg tool_baud_rate)"
-      tool_stop_bits="$(arg tool_stop_bits)"
-      tool_rx_idle_chars="$(arg tool_rx_idle_chars)"
-      tool_tx_idle_chars="$(arg tool_tx_idle_chars)"
       tool_device_name="$(arg tool_device_name)"
-      tool_tcp_port="$(arg tool_tcp_port)"
       robot_ip="$(arg robot_ip)"
       script_filename="$(arg script_filename)"
@@ -81,8 +62,4 @@
       input_recipe_filename="$(arg input_recipe_filename)"
       reverse_ip="$(arg reverse_ip)"
-      script_command_port="$(arg script_command_port)"
-      reverse_port="$(arg reverse_port)"
-      script_sender_port="$(arg script_sender_port)"
-      trajectory_port="$(arg trajectory_port)"
     >
       <!-- position robot in the world -->
@@ -91,5 +68,5 @@
     <xacro:if value="$(arg sim_gazebo)">
       <!-- Gazebo plugins -->
-      <gazebo reference="ur_base"/>
+      <gazebo reference="${parent}"/>
       <gazebo>
         <plugin filename="libgazebo_ros2_control.so" name="gazebo_ros2_control">
@@ -100,5 +77,5 @@
     <xacro:if value="$(arg sim_ignition)">
       <!-- Gazebo plugins -->
-      <gazebo reference="ur_base"/>
+      <gazebo reference="${parent}"/>
       <gazebo>
         <plugin filename="libign_ros2_control-system.so" name="ign_ros2_control::IgnitionROS2ControlPlugin">
