Commit message: DEL: removed world frame in favour of ur_base

File: aegis_description/urdf/aegis.urdf.xacro (robot description, xacro)
@@ -2,5 +2,5 @@
 <robot xmlns:xacro="http://wiki.ros.org/xacro" name="aegis">
   <xacro:arg name="mock_hardware" default="false"/>
-  <xacro:arg name="base_link" default="world"/>
+  <xacro:arg name="base_link" default="ur_base"/>
   <xacro:arg name="prefix" default=""/>
   <xacro:arg name="tf_prefix" default=""/>

File: aegis_description/urdf/aegis.xacro (robot description, xacro)
@@ -15,5 +15,5 @@
   <xacro:macro name="aegis_robot" params="parent tf_prefix prefix mock_hardware">
     <xacro:ur_definition name="aegis" parent="${parent}" tf_prefix="${tf_prefix}" mock_hardware="${mock_hardware}"/>
-    <xacro:cell parent="ur_base"/>
+    <xacro:cell parent="${parent}"/>
     <xacro:adapter_to_sensor parent="tool0" prefix="${prefix}"/>
     <xacro:ft_sensor_schunk_axia80 parent="adapter_to_sensor_end" prefix="${prefix}" mock_hardware="${mock_hardware}"/>

File: aegis_description/urdf/modules/cell.xacro (robot description, xacro)
@@ -4,5 +4,5 @@
     <joint name="ur_base_to_cell" type="fixed">
       <origin xyz="0 0 -0.806" rpy="0 0 -${0.5 * pi}"/>
-      <parent link="ur_base"/>
+      <parent link="${parent}"/>
       <child link="cell"/>
     </joint>
@@ -63,5 +63,4 @@
       </collision>
     </link>
-    <link name="ur_base"/>
   </xacro:macro>
 </robot>

File: aegis_description/urdf/modules/ur_definition.xacro (robot description, xacro)
@@ -5,10 +5,4 @@
   <!-- Descriptions of the arguments can be found in the <ur_robot_driver>/src/hardware_interface.cpp file -->
   <xacro:macro name="ur_definition" params="name parent tf_prefix mock_hardware">
-    <!-- For simulation, the global parent must be the same as ur_base -->
-    <joint name="world_to_ur_base" type="fixed">
-      <origin xyz="0 0 0" rpy="0 0 0"/>
-      <parent link="${parent}"/>
-      <child link="ur_base"/>
-    </joint>
     <!-- parameters -->
     <xacro:arg name="tf_prefix" default="${tf_prefix}"/>
@@ -46,5 +40,5 @@
       name="${name}"
       tf_prefix="$(arg tf_prefix)"
-      parent="ur_base"
+      parent="${parent}"
       joint_limits_parameters_file="$(arg joint_limit_params)"
       kinematics_parameters_file="$(arg kinematics_calibration)"
@@ -69,5 +63,5 @@
       reverse_ip="$(arg reverse_ip)"
     >
-      <!-- position robot in the world -->
+      <!-- robot relative pose -->
       <origin xyz="0 0 0" rpy="0 0 0"/>
     </xacro:ur_robot>

Commit message: Add parameter to disable cell

File: aegis_description/urdf/aegis.urdf.xacro (robot description, xacro)
@@ -2,4 +2,5 @@
 <robot xmlns:xacro="http://wiki.ros.org/xacro" name="aegis">
   <xacro:arg name="mock_hardware" default="false"/>
+  <xacro:arg name="disable_cell" default="false"/>
   <xacro:arg name="base_link" default="world"/>
   <xacro:arg name="prefix" default=""/>
@@ -7,4 +8,4 @@
   <xacro:include filename="$(find aegis_description)/urdf/aegis.xacro"/>
   <link name="$(arg base_link)"/>
-  <xacro:aegis_robot parent="$(arg base_link)" tf_prefix="$(arg tf_prefix)" prefix="$(arg prefix)" mock_hardware="$(arg mock_hardware)"/>
+  <xacro:aegis_robot parent="$(arg base_link)" tf_prefix="$(arg tf_prefix)" prefix="$(arg prefix)" mock_hardware="$(arg mock_hardware)" disable_cell="$(arg disable_cell)"/>
 </robot>

File: aegis_description/urdf/aegis.xacro (robot description, xacro)
@@ -13,6 +13,8 @@
   <xacro:include filename="$(find aegis_description)/urdf/modules/camera_tool_basler.xacro"/>
   <xacro:include filename="$(find aegis_description)/urdf/modules/lens_computar.xacro"/>
-  <xacro:macro name="aegis_robot" params="parent tf_prefix prefix mock_hardware">
-    <xacro:cell parent="${parent}"/>
+  <xacro:macro name="aegis_robot" params="parent tf_prefix prefix mock_hardware disable_cell">
+    <xacro:unless value="${disable_cell}">
+      <xacro:cell parent="${parent}"/>
+    </xacro:unless>
     <xacro:ur_definition name="aegis" parent="${parent}" tf_prefix="${tf_prefix}" mock_hardware="${mock_hardware}"/>
     <xacro:adapter_to_sensor parent="tool0" prefix="${prefix}"/>

Commit message: Add parameter to disable cell collision

File: aegis_description/urdf/aegis.urdf.xacro (robot description, xacro)
@@ -3,4 +3,5 @@
   <xacro:arg name="mock_hardware" default="false"/>
   <xacro:arg name="disable_cell" default="false"/>
+  <xacro:arg name="disable_cell_collision" default="false"/>
   <xacro:arg name="base_link" default="world"/>
   <xacro:arg name="prefix" default=""/>
@@ -8,4 +9,11 @@
   <xacro:include filename="$(find aegis_description)/urdf/aegis.xacro"/>
   <link name="$(arg base_link)"/>
-  <xacro:aegis_robot parent="$(arg base_link)" tf_prefix="$(arg tf_prefix)" prefix="$(arg prefix)" mock_hardware="$(arg mock_hardware)" disable_cell="$(arg disable_cell)"/>
+  <xacro:aegis_robot
+    parent="$(arg base_link)"
+    tf_prefix="$(arg tf_prefix)"
+    prefix="$(arg prefix)"
+    mock_hardware="$(arg mock_hardware)"
+    disable_cell="$(arg disable_cell)"
+    disable_cell_collision="$(arg disable_cell_collision)"
+  />
 </robot>

File: aegis_description/urdf/aegis.xacro (robot description, xacro)
@@ -13,7 +13,7 @@
   <xacro:include filename="$(find aegis_description)/urdf/modules/camera_tool_basler.xacro"/>
   <xacro:include filename="$(find aegis_description)/urdf/modules/lens_computar.xacro"/>
-  <xacro:macro name="aegis_robot" params="parent tf_prefix prefix mock_hardware disable_cell">
+  <xacro:macro name="aegis_robot" params="parent tf_prefix prefix mock_hardware disable_cell disable_cell_collision">
     <xacro:unless value="${disable_cell}">
-      <xacro:cell parent="${parent}"/>
+      <xacro:cell parent="${parent}" disable_cell_collision="${disable_cell_collision}"/>
     </xacro:unless>
     <xacro:ur_definition name="aegis" parent="${parent}" tf_prefix="${tf_prefix}" mock_hardware="${mock_hardware}"/>

File: aegis_description/urdf/modules/cell.xacro (robot description, xacro)
@@ -1,5 +1,5 @@
 <?xml version="1.0"?>
 <robot xmlns:xacro="http://ros.org/wiki/xacro">
-  <xacro:macro name="cell" params="parent">
+  <xacro:macro name="cell" params="parent disable_cell_collision">
     <joint name="world_to_cell" type="fixed">
       <origin xyz="0 0 -0.806" rpy="0 0 -${0.5 * pi}"/>
@@ -14,52 +14,54 @@
         </geometry>
       </visual>
-      <collision>
-        <origin xyz="0 -0.162 0.435" rpy="0 0 0"/>
-        <geometry>
-          <box size="0.72 0.324 0.87"/>
-        </geometry>
-      </collision>
-      <collision>
-        <origin xyz="0 0.162 0.41" rpy="0 0 0"/>
-        <geometry>
-          <box size="0.72 0.324 0.82"/>
-        </geometry>
-      </collision>
-      <collision>
-        <origin xyz="0.48 0 0.97" rpy="0 0 0"/>
-        <geometry>
-          <box size="0.08 0.648 1.94"/>
-        </geometry>
-      </collision>
-      <collision>
-        <origin xyz="0.4 0 0.435" rpy="0 0 0"/>
-        <geometry>
-          <box size="0.08 0.648 0.87"/>
-        </geometry>
-      </collision>
-      <collision>
-        <origin xyz="-0.48 0 0.97" rpy="0 0 0"/>
-        <geometry>
-          <box size="0.08 0.648 1.94"/>
-        </geometry>
-      </collision>
-      <collision>
-        <origin xyz="-0.4 0 0.435" rpy="0 0 0"/>
-        <geometry>
-          <box size="0.08 0.648 0.87"/>
-        </geometry>
-      </collision>
-      <collision>
-        <origin xyz="0 0.04 1.98" rpy="0 0 0"/>
-        <geometry>
-          <box size="1.04 0.728 0.08"/>
-        </geometry>
-      </collision>
-      <collision>
-        <origin xyz="0 -0.62 1.2" rpy="0 0 0"/>
-        <geometry>
-          <box size="2.4 0.02 2.4"/>
-        </geometry>
-      </collision>
+      <xacro:unless value="${disable_cell_collision}">
+        <collision>
+          <origin xyz="0 -0.162 0.435" rpy="0 0 0"/>
+          <geometry>
+            <box size="0.72 0.324 0.87"/>
+          </geometry>
+        </collision>
+        <collision>
+          <origin xyz="0 0.162 0.41" rpy="0 0 0"/>
+          <geometry>
+            <box size="0.72 0.324 0.82"/>
+          </geometry>
+        </collision>
+        <collision>
+          <origin xyz="0.48 0 0.97" rpy="0 0 0"/>
+          <geometry>
+            <box size="0.08 0.648 1.94"/>
+          </geometry>
+        </collision>
+        <collision>
+          <origin xyz="0.4 0 0.435" rpy="0 0 0"/>
+          <geometry>
+            <box size="0.08 0.648 0.87"/>
+          </geometry>
+        </collision>
+        <collision>
+          <origin xyz="-0.48 0 0.97" rpy="0 0 0"/>
+          <geometry>
+            <box size="0.08 0.648 1.94"/>
+          </geometry>
+        </collision>
+        <collision>
+          <origin xyz="-0.4 0 0.435" rpy="0 0 0"/>
+          <geometry>
+            <box size="0.08 0.648 0.87"/>
+          </geometry>
+        </collision>
+        <collision>
+          <origin xyz="0 0.04 1.98" rpy="0 0 0"/>
+          <geometry>
+            <box size="1.04 0.728 0.08"/>
+          </geometry>
+        </collision>
+        <collision>
+          <origin xyz="0 -0.62 1.2" rpy="0 0 0"/>
+          <geometry>
+            <box size="2.4 0.02 2.4"/>
+          </geometry>
+        </collision>
+      </xacro:unless>
     </link>
   </xacro:macro>
