Commit message: Changed URDF related launch arguments to prefix `model_*`

File: aegis_description/urdf/aegis.urdf.xacro (robot description, xacro)
@@ -4,5 +4,5 @@
   <xacro:arg name="disable_cell" default="false"/>
   <xacro:arg name="disable_cell_collision" default="false"/>
-  <xacro:arg name="disable_leds" default="false"/>
+  <xacro:arg name="disable_led_supports" default="false"/>
   <xacro:arg name="base_link" default="world"/>
   <xacro:arg name="prefix" default=""/>
@@ -17,5 +17,5 @@
     disable_cell="$(arg disable_cell)"
     disable_cell_collision="$(arg disable_cell_collision)"
-    disable_leds="$(arg disable_leds)"
+    disable_led_supports="$(arg disable_led_supports)"
   />
 </robot>

File: aegis_description/urdf/aegis.xacro (robot description, xacro)
@@ -16,6 +16,6 @@
   <xacro:include filename="$(find aegis_description)/urdf/modules/camera_tool_basler.xacro"/>
   <xacro:include filename="$(find aegis_description)/urdf/modules/lens_computar.xacro"/>
-  <xacro:macro name="aegis_robot" params="parent tf_prefix prefix mock_hardware disable_cell disable_cell_collision disable_leds">
-    <xacro:cell parent="${parent}" disable_cell="${disable_cell}" disable_cell_collision="${disable_cell_collision}" disable_leds="${disable_leds}"/>
+  <xacro:macro name="aegis_robot" params="parent tf_prefix prefix mock_hardware disable_cell disable_cell_collision disable_led_supports">
+    <xacro:cell parent="${parent}" disable_cell="${disable_cell}" disable_cell_collision="${disable_cell_collision}" disable_led_supports="${disable_led_supports}"/>
     <xacro:adapter_cell parent="${parent}" prefix="${prefix}" disable_cell="${disable_cell}" disable_cell_collision="${disable_cell_collision}"/>
     <xacro:ur_definition name="aegis" parent="${parent}" tf_prefix="${tf_prefix}" mock_hardware="${mock_hardware}"/>

File: aegis_description/urdf/modules/cell.xacro (robot description, xacro)
@@ -1,5 +1,5 @@
 <?xml version="1.0"?>
 <robot xmlns:xacro="http://ros.org/wiki/xacro">
-  <xacro:macro name="cell" params="parent disable_cell disable_cell_collision disable_leds">
+  <xacro:macro name="cell" params="parent disable_cell disable_cell_collision disable_led_supports">
     <xacro:unless value="${disable_cell}">
       <joint name="world_to_cell" type="fixed">
@@ -66,7 +66,7 @@
         </xacro:unless>
       </link>
-      <xacro:unless value="${disable_leds}">
-      <xacro:lighting_support_right parent="cell" prefix="" disable_cell_collision="${disable_cell_collision}"/>
-      <xacro:lighting_support_left parent="cell" prefix="" disable_cell_collision="${disable_cell_collision}"/>
+      <xacro:unless value="${disable_led_supports}">
+        <xacro:lighting_support_right parent="cell" prefix="" disable_cell_collision="${disable_cell_collision}"/>
+        <xacro:lighting_support_left parent="cell" prefix="" disable_cell_collision="${disable_cell_collision}"/>
       </xacro:unless>
     </xacro:unless>
