Commit message: working robot_description launch

File: aegis_description/urdf/aegis.xacro (robot description, xacro)
@@ -6,6 +6,6 @@
   <xacro:include filename="$(find aegis_description)/urdf/modules/adapter_from_sensor.xacro"/>
   <xacro:include filename="$(find robotiq_hande_description)/urdf/robotiq_hande_gripper.xacro"/>
-  <xacro:macro name="aegis_robot" params="parent prefix kinematics_calibration mock_hardware">
-    <xacro:ur_definition name="aegis" parent="${parent}" prefix="${prefix}" kinematics_calibration="${kinematics_calibration}" mock_hardware="${mock_hardware}"/>
+  <xacro:macro name="aegis_robot" params="parent prefix mock_hardware">
+    <xacro:ur_definition name="aegis" parent="${parent}" prefix="${prefix}" mock_hardware="${mock_hardware}"/>
     <xacro:adapter_to_sensor parent="tool0" prefix="${prefix}"/>
     <xacro:ft_sensor_schunk_axia80 parent="adapter_to_sensor_end" prefix="${prefix}" mock_hardware="${mock_hardware}"/>

Commit message: WIP: configure urdf for basler

File: aegis_description/urdf/aegis.xacro (robot description, xacro)
@@ -8,4 +8,5 @@
   <xacro:include filename="$(find aegis_description)/urdf/modules/adapter_from_sensor.xacro"/>
   <xacro:include filename="$(find aegis_description)/urdf/modules/robotiq_hande_gripper.xacro"/>
+  <xacro:include filename="$(find aegis_description)/urdf/modules/basler_camera_mounting.xacro"/>
   <xacro:macro name="aegis_robot" params="parent tf_prefix prefix mock_hardware">
     <xacro:cell parent="${parent}"/>
@@ -16,4 +17,5 @@
     <xacro:adapter_from_sensor parent="tool_mount_link" prefix="${prefix}"/>
     <xacro:hande_gripper parent="adapter_from_sensor_end" prefix="${prefix}" mock_hardware="${mock_hardware}"/>
+    <xacro:basler_camera_mounting parent="adapter_to_camera_mounting_back" prefix="${prefix}"/>
   </xacro:macro>
 </robot>

File: aegis_description/urdf/modules/adapter_to_sensor.xacro (robot description, xacro)
@@ -46,4 +46,10 @@
     </joint>
     <link name="${prefix}adapter_to_sensor_end"/>
+    <joint name="${prefix}adapter_to_camera_mounting_back_joint" type="fixed">
+      <origin xyz="0 ${radius2} 0" rpy="0 0 0"/>
+      <parent link="${prefix}adapter_to_sensor"/>
+      <child link="${prefix}adapter_to_camera_mounting_back"/>
+    </joint>
+    <link name="${prefix}adapter_to_camera_mounting_back"/>
   </xacro:macro>
 </robot>

Commit message: WIP: replace sensor_to adepter with our custom part

File: aegis_description/urdf/aegis.xacro (robot description, xacro)
@@ -18,4 +18,5 @@
     <xacro:hande_gripper parent="adapter_from_sensor_end" prefix="${prefix}" mock_hardware="${mock_hardware}"/>
     <xacro:basler_camera_mounting parent="adapter_to_camera_mounting_back" prefix="${prefix}"/>
+    <!-- <xacro:basler_camera_mounting parent="adapter_to_camera_mounting_front" prefix="${prefix}"/> -->
   </xacro:macro>
 </robot>

File: aegis_description/urdf/modules/adapter_to_sensor.xacro (robot description, xacro)
@@ -15,7 +15,7 @@
     <link name="${prefix}adapter_to_sensor">
       <visual>
-        <origin xyz="0 0 ${0.5 * height1}" rpy="0 0 0"/>
+        <origin xyz="0 0 0.021" rpy="0 ${pi} ${pi}"/>
         <geometry>
-          <cylinder radius="${radius1}" length="${height1}"/>
+           <mesh filename="package://aegis_description/meshes/adapter_to_sensor.dae" scale="0.001 0.001 0.001"/>
         </geometry>
         <material name="black">
@@ -23,5 +23,5 @@
         </material>
       </visual>
-      <visual>
+      <!-- <visual>
         <origin xyz="0 0 ${height1 + 0.5 * height2}" rpy="0 0 0"/>
         <geometry>
@@ -31,5 +31,5 @@
           <color rgba="0.04 0.04 0.04 1"/>
         </material>
-      </visual>
+      </visual> -->
       <xacro:cylinders_inertial r1="${radius1}" l1="${height1}" r2="${radius2}" l2="${height2}" m="${mass}"/>
       <collision>
@@ -47,9 +47,15 @@
     <link name="${prefix}adapter_to_sensor_end"/>
     <joint name="${prefix}adapter_to_camera_mounting_back_joint" type="fixed">
-      <origin xyz="0 ${radius2} 0" rpy="0 0 0"/>
+      <origin xyz="0 ${radius2} 0" rpy="0 ${pi} 0"/>
       <parent link="${prefix}adapter_to_sensor"/>
       <child link="${prefix}adapter_to_camera_mounting_back"/>
     </joint>
     <link name="${prefix}adapter_to_camera_mounting_back"/>
+    <joint name="${prefix}adapter_to_camera_mounting_front_joint" type="fixed">
+      <origin xyz="0 ${radius2} 0" rpy="0 ${pi} 0"/>
+      <parent link="${prefix}adapter_to_sensor"/>
+      <child link="${prefix}adapter_to_camera_mounting_front"/>
+    </joint>
+    <link name="${prefix}adapter_to_camera_mounting_front"/>
   </xacro:macro>
 </robot>

File: aegis_description/urdf/modules/basler_camera_mounting.xacro (robot description, xacro)
@@ -17,5 +17,5 @@
         <origin xyz="0 0 0" rpy="0 0 0"/>
         <geometry>
-          <mesh filename="package://aegis_description/meshes/basler_camera_mounting.dae" scale="1.0 1.0 1.0"/>
+          <mesh filename="package://aegis_description/meshes/basler_camera_mounting.dae" scale="0.001 0.001 0.001"/>
         </geometry>
       </visual>

Commit message: ADD: front and back camera mounting

File: aegis_description/urdf/aegis.xacro (robot description, xacro)
@@ -17,6 +17,6 @@
     <xacro:adapter_from_sensor parent="tool_mount_link" prefix="${prefix}"/>
     <xacro:hande_gripper parent="adapter_from_sensor_end" prefix="${prefix}" mock_hardware="${mock_hardware}"/>
-    <xacro:basler_camera_mounting parent="adapter_to_camera_mounting_back" prefix="${prefix}"/>
-    <!-- <xacro:basler_camera_mounting parent="adapter_to_camera_mounting_front" prefix="${prefix}"/> -->
+    <xacro:basler_camera_mounting parent="adapter_to_camera_mounting_back" prefix="${prefix}" side="back"/>
+    <xacro:basler_camera_mounting parent="adapter_to_camera_mounting_front" prefix="${prefix}" side="front"/>
   </xacro:macro>
 </robot>

File: aegis_description/urdf/modules/basler_camera_mounting.xacro (robot description, xacro)
@@ -2,5 +2,5 @@
 <robot xmlns:xacro="http://ros.org/wiki/xacro">
   <!-- <xacro:include filename="$(find aegis_description)/urdf/cylinders_inertial.xacro"/> -->
-  <xacro:macro name="basler_camera_mounting" params="prefix parent">
+  <xacro:macro name="basler_camera_mounting" params="prefix parent side">
     <xacro:property name="mass" value="0.217"/>
     <xacro:property name="mounting_width" value="0.07002"/>
@@ -8,10 +8,10 @@
     <!-- <xacro:property name="radius2" value="0.0315"/>
     <xacro:property name="height2" value="0.007"/> -->
-    <joint name="basler_camera_mounting_joint" type="fixed">
+    <joint name="basler_camera_mounting_joint_${side}" type="fixed">
       <origin xyz="0 0 ${0.5 * mounting_height}" rpy="0 0 0"/>
       <parent link="${parent}"/>
-      <child link="${prefix}basler_camera_mounting"/>
+      <child link="${prefix}basler_camera_mounting_${side}"/>
     </joint>
-    <link name="${prefix}basler_camera_mounting">
+    <link name="${prefix}basler_camera_mounting_${side}">
       <visual>
         <origin xyz="0 0 0" rpy="0 0 0"/>

Commit message: ADD: prcise basler camera position with two cameras

File: aegis_description/urdf/aegis.xacro (robot description, xacro)
@@ -9,4 +9,5 @@
   <xacro:include filename="$(find aegis_description)/urdf/modules/robotiq_hande_gripper.xacro"/>
   <xacro:include filename="$(find aegis_description)/urdf/modules/basler_camera_mounting.xacro"/>
+  <xacro:include filename="$(find aegis_description)/urdf/modules/basler_camera.xacro"/>
   <xacro:macro name="aegis_robot" params="parent tf_prefix prefix mock_hardware">
     <xacro:cell parent="${parent}"/>
@@ -19,4 +20,6 @@
     <xacro:basler_camera_mounting parent="adapter_to_camera_mounting_back" prefix="${prefix}" side="back"/>
     <xacro:basler_camera_mounting parent="adapter_to_camera_mounting_front" prefix="${prefix}" side="front"/>
+    <xacro:basler_camera parent="mounting_to_camera_back" prefix="${prefix}" side="back"/>
+    <xacro:basler_camera parent="mounting_to_camera_front" prefix="${prefix}" side="front"/>
   </xacro:macro>
 </robot>

File: aegis_description/urdf/modules/adapter_to_sensor.xacro (robot description, xacro)
@@ -10,5 +10,5 @@
     <xacro:property name="height_to_adapter" value="0.01456"/>
     <xacro:property name="height_total" value="0.02080"/>
-    <xacro:property name="width" value="0.08580"/>
+    <xacro:property name="width" value="0.0860"/>
     <joint name="${prefix}adapter_to_sensor_joint" type="fixed">
       <origin xyz="0 0 0" rpy="0 0 0"/>

File: aegis_description/urdf/modules/basler_camera_mounting.xacro (robot description, xacro)
@@ -4,8 +4,16 @@
   <xacro:macro name="basler_camera_mounting" params="prefix parent side">
     <xacro:property name="mass" value="0.217"/>
-    <xacro:property name="mounting_width" value="0.07002"/>
+    <xacro:property name="mounting_width" value="0.07000"/>
     <xacro:property name="mounting_height" value="0.001353"/>
+    <!-- <xacro:property name="mounting_insert_depth" value="0.0076"/> -->
     <!-- <xacro:property name="radius2" value="0.0315"/>
     <xacro:property name="height2" value="0.007"/> -->
+    <!-- <xacro:property name="mounting_dist_a" value="0.09070"/>
+    <xacro:property name="mounting_dist_b" value="-0.0460"/>
+    <xacro:property name="mounting_dist_c_x" value="-0.03471"/>
+    <xacro:property name="mounting_dist_c_z" value="-0.04136"/> -->
+    <xacro:property name="mounting_yaw" value="-0.6981"/>
+    <xacro:property name="mounting_dist_z" value="-0.06607"/>
+    <xacro:property name="mounting_dist_x" value="0.119084"/>
     <joint name="basler_camera_mounting_joint_${side}" type="fixed">
       <origin xyz="0 0 ${0.5 * mounting_height}" rpy="0 0 0"/>
@@ -33,4 +41,12 @@
     </joint>
     <link name="${prefix}adapter_from_sensor_end"/> -->
+    <joint name="${prefix}mounting_to_camera_${side}_joint" type="fixed">
+      <origin
+        xyz="${mounting_dist_x} 0 ${mounting_dist_z}"
+        rpy="${mounting_yaw} 0 ${-0.5 * pi}"/>
+      <parent link="${prefix}basler_camera_mounting_${side}"/>
+      <child link="${prefix}mounting_to_camera_${side}"/>
+    </joint>
+    <link name="${prefix}mounting_to_camera_${side}"/>
   </xacro:macro>
 </robot>

Commit message: ADD: separate component for camera lens

File: aegis_description/urdf/aegis.xacro (robot description, xacro)
@@ -10,4 +10,5 @@
   <xacro:include filename="$(find aegis_description)/urdf/modules/basler_camera_mounting.xacro"/>
   <xacro:include filename="$(find aegis_description)/urdf/modules/basler_camera.xacro"/>
+  <xacro:include filename="$(find aegis_description)/urdf/modules/computar_lens.xacro"/>
   <xacro:macro name="aegis_robot" params="parent tf_prefix prefix mock_hardware">
     <xacro:cell parent="${parent}"/>
@@ -22,4 +23,6 @@
     <xacro:basler_camera parent="mounting_to_camera_back" prefix="${prefix}" side="back"/>
     <xacro:basler_camera parent="mounting_to_camera_front" prefix="${prefix}" side="front"/>
+    <xacro:computar_lens parent="camera_to_lens_back" prefix="${prefix}" side="back"/>
+    <xacro:computar_lens parent="camera_to_lens_front" prefix="${prefix}" side="front"/>
   </xacro:macro>
 </robot>

File: aegis_description/urdf/modules/basler_camera.xacro (robot description, xacro)
@@ -23,13 +23,4 @@
         </geometry>
       </visual>
-      <visual>
-        <origin xyz="0 0 ${lens_offset}" rpy="0 0 ${pi}"/>
-        <geometry>
-          <cylinder radius="${lens_radius}" length="${lens_height}"/>
-        </geometry>
-        <material name="black">
-          <color rgba="0.04 0.04 0.04 1"/>
-        </material>
-      </visual>
       <!-- <xacro:cylinders_inertial r1="${radius1}" l1="${height1}" r2="${radius2}" l2="${height2}" m="${mass}"/> -->
       <collision>
@@ -39,11 +30,11 @@
         </geometry>
       </collision>
-      <collision>
-        <origin xyz="0 0 ${lens_offset}" rpy="0 0 ${pi}"/>
-        <geometry>
-          <cylinder radius="${lens_radius}" length="${lens_height}"/>
-        </geometry>
-      </collision>
     </link>
+    <joint name="${prefix}camera_to_lens_${side}_joint" type="fixed">
+      <origin xyz="0 0 ${lens_offset}" rpy="0 0 0"/>
+      <parent link="${prefix}basler_camera_${side}"/>
+      <child link="${prefix}camera_to_lens_${side}"/>
+    </joint>
+    <link name="${prefix}camera_to_lens_${side}"/>
   </xacro:macro>
 </robot>

Commit message: Integrate mounted OAK-D SR tool camera into Aegis Xacro model

File: aegis_description/urdf/aegis.xacro (robot description, xacro)
@@ -2,5 +2,4 @@
 <robot xmlns:xacro="http://wiki.ros.org/xacro">
   <xacro:include filename="$(find aegis_description)/urdf/modules/cell.xacro"/>
-  <xacro:include filename="$(find aegis_description)/urdf/modules/luxonis_oakd_pro_scene.xacro"/>
   <xacro:include filename="$(find aegis_description)/urdf/modules/ur_definition.xacro"/>
   <xacro:include filename="$(find aegis_description)/urdf/modules/adapter_to_sensor.xacro"/>
@@ -8,4 +7,7 @@
   <xacro:include filename="$(find aegis_description)/urdf/modules/adapter_from_sensor.xacro"/>
   <xacro:include filename="$(find aegis_description)/urdf/modules/robotiq_hande_gripper.xacro"/>
+  <xacro:include filename="$(find aegis_description)/urdf/modules/luxonis_oakd_pro_scene.xacro"/>
+  <xacro:include filename="$(find aegis_description)/urdf/modules/mount_camera_tool_luxonis.xacro"/>
+  <xacro:include filename="$(find aegis_description)/urdf/modules/camera_tool_luxonis.xacro"/>
   <xacro:include filename="$(find aegis_description)/urdf/modules/basler_camera_mounting.xacro"/>
   <xacro:include filename="$(find aegis_description)/urdf/modules/basler_camera.xacro"/>
@@ -13,5 +15,4 @@
   <xacro:macro name="aegis_robot" params="parent tf_prefix prefix mock_hardware">
     <xacro:cell parent="${parent}"/>
-    <xacro:luxonis_oakd_pro_scene parent="cell"/>
     <xacro:ur_definition name="aegis" parent="ur_base" tf_prefix="${tf_prefix}" mock_hardware="${mock_hardware}"/>
     <xacro:adapter_to_sensor parent="tool0" prefix="${prefix}"/>
@@ -19,4 +20,7 @@
     <xacro:adapter_from_sensor parent="tool_mount_link" prefix="${prefix}"/>
     <xacro:hande_gripper parent="adapter_from_sensor_end" prefix="${prefix}" mock_hardware="${mock_hardware}"/>
+    <xacro:luxonis_oakd_pro_scene parent="cell"/>
+    <xacro:mount_camera_tool_luxonis parent="mount" prefix="${prefix}"/>
+    <xacro:camera_tool_luxonis parent="camera_tool" prefix="${prefix}"/>
     <xacro:basler_camera_mounting parent="adapter_to_camera_mounting_back" prefix="${prefix}" side="back"/>
     <xacro:basler_camera_mounting parent="adapter_to_camera_mounting_front" prefix="${prefix}" side="front"/>

File: aegis_description/urdf/modules/adapter_to_sensor.xacro (robot description, xacro)
@@ -52,4 +52,10 @@
     </joint>
     <link name="${prefix}adapter_to_camera_mounting_front"/>
+    <joint name="adapter_to_mount_joint" type="fixed">
+      <origin xyz="0 0 ${height_to_adapter}" rpy="0 ${pi} ${pi / 2}"/>
+      <parent link="${prefix}adapter_to_sensor"/>
+      <child link="${prefix}mount"/>
+    </joint>
+    <link name="${prefix}mount"/>
   </xacro:macro>
 </robot>

Commit message: Add OAK-D SR tool camera to DepthAI launch setup

File: aegis_description/urdf/aegis.xacro (robot description, xacro)
@@ -7,5 +7,5 @@
   <xacro:include filename="$(find aegis_description)/urdf/modules/adapter_from_sensor.xacro"/>
   <xacro:include filename="$(find aegis_description)/urdf/modules/robotiq_hande_gripper.xacro"/>
-  <xacro:include filename="$(find aegis_description)/urdf/modules/luxonis_oakd_pro_scene.xacro"/>
+  <xacro:include filename="$(find aegis_description)/urdf/modules/camera_scene_luxonis.xacro"/>
   <xacro:include filename="$(find aegis_description)/urdf/modules/mount_camera_tool_luxonis.xacro"/>
   <xacro:include filename="$(find aegis_description)/urdf/modules/camera_tool_luxonis.xacro"/>
@@ -20,5 +20,5 @@
     <xacro:adapter_from_sensor parent="tool_mount_link" prefix="${prefix}"/>
     <xacro:hande_gripper parent="adapter_from_sensor_end" prefix="${prefix}" mock_hardware="${mock_hardware}"/>
-    <xacro:luxonis_oakd_pro_scene parent="cell"/>
+    <xacro:camera_scene_luxonis parent="cell"/>
     <xacro:mount_camera_tool_luxonis parent="mount" prefix="${prefix}"/>
     <xacro:camera_tool_luxonis parent="camera_tool" prefix="${prefix}"/>

File: aegis_description/urdf/modules/camera_scene_luxonis.xacro (robot description, xacro)
@@ -1,10 +1,10 @@
 <?xml version="1.0"?>
 <robot xmlns:xacro="http://ros.org/wiki/xacro">
-  <xacro:arg name="scene_camera_name" default="oak_d_pro_scene"/>
+  <xacro:arg name="scene_camera_name" default="cam_scene"/>
   <xacro:arg name="scene_camera_model" default="OAK-D-S2"/>
-  <xacro:arg name="scene_camera_base_frame" default="oak_d_pro_scene_frame"/>
+  <xacro:arg name="scene_camera_base_frame" default="cam_scene_frame"/>
   <xacro:arg name="scene_camera_rs_compat" default="false"/>
   <xacro:include filename="$(find depthai_descriptions)/urdf/include/depthai_macro.urdf.xacro"/>
-  <xacro:macro name="luxonis_oakd_pro_scene" params="parent">
+  <xacro:macro name="camera_scene_luxonis" params="parent">
     <xacro:depthai_camera
       camera_name="$(arg scene_camera_name)"

File: aegis_description/urdf/modules/camera_tool_luxonis.xacro (robot description, xacro)
@@ -1,7 +1,7 @@
 <?xml version="1.0"?>
 <robot xmlns:xacro="http://ros.org/wiki/xacro">
-  <xacro:arg name="tool_camera_name" default="oak_d_sr"/>
+  <xacro:arg name="tool_camera_name" default="cam_tool"/>
   <xacro:arg name="tool_camera_model" default="OAK-D-SR-POE"/>
-  <xacro:arg name="tool_camera_base_frame" default="oak_d_sr_tool_frame"/>
+  <xacro:arg name="tool_camera_base_frame" default="cam_tool_frame"/>
   <xacro:arg name="tool_camera_rs_compat" default="false"/>
   <xacro:include filename="$(find depthai_descriptions)/urdf/include/depthai_macro.urdf.xacro"/>
@@ -16,5 +16,5 @@
       cam_pos_z="-0.039"
       cam_roll="0"
-      cam_pitch="${pi/2}"
+      cam_pitch="${pi / 2}"
       cam_yaw="0"
       rs_compat="$(arg tool_camera_rs_compat)"
