Commit message: CHG: naming convention

File: aegis_description/urdf/aegis.xacro (robot description, xacro)
@@ -8,7 +8,7 @@
   <xacro:include filename="$(find aegis_description)/urdf/modules/adapter_from_sensor.xacro"/>
   <xacro:include filename="$(find aegis_description)/urdf/modules/robotiq_hande_gripper.xacro"/>
-  <xacro:include filename="$(find aegis_description)/urdf/modules/basler_camera_mounting.xacro"/>
-  <xacro:include filename="$(find aegis_description)/urdf/modules/basler_camera.xacro"/>
-  <xacro:include filename="$(find aegis_description)/urdf/modules/computar_lens.xacro"/>
+  <xacro:include filename="$(find aegis_description)/urdf/modules/mount_camera_tool_basler.xacro"/>
+  <xacro:include filename="$(find aegis_description)/urdf/modules/camera_tool_basler.xacro"/>
+  <xacro:include filename="$(find aegis_description)/urdf/modules/lens_computar.xacro"/>
   <xacro:macro name="aegis_robot" params="parent tf_prefix prefix mock_hardware">
     <xacro:cell parent="${parent}"/>
@@ -19,10 +19,10 @@
     <xacro:adapter_from_sensor parent="tool_mount_link" prefix="${prefix}"/>
     <xacro:hande_gripper parent="adapter_from_sensor_end" prefix="${prefix}" mock_hardware="${mock_hardware}"/>
-    <xacro:basler_camera_mounting parent="adapter_to_camera_mounting_back" prefix="${prefix}" side="back"/>
-    <xacro:basler_camera_mounting parent="adapter_to_camera_mounting_front" prefix="${prefix}" side="front"/>
-    <xacro:basler_camera parent="mounting_to_camera_back" prefix="${prefix}" side="back"/>
-    <xacro:basler_camera parent="mounting_to_camera_front" prefix="${prefix}" side="front"/>
-    <xacro:computar_lens parent="camera_to_lens_back" prefix="${prefix}" side="back"/>
-    <xacro:computar_lens parent="camera_to_lens_front" prefix="${prefix}" side="front"/>
+    <xacro:mount_camera_tool_balser parent="adapter_to_mount_camera_tool_right" prefix="${prefix}" side="right"/>
+    <xacro:mount_camera_tool_balser parent="adapter_to_mount_camera_tool_left" prefix="${prefix}" side="left"/>
+    <xacro:camera_tool_basler parent="mount_to_camera_right" prefix="${prefix}" side="right"/>
+    <xacro:camera_tool_basler parent="mount_to_camera_left" prefix="${prefix}" side="left"/>
+    <xacro:lens_computar parent="camera_to_lens_right" prefix="${prefix}" side="right"/>
+    <xacro:lens_computar parent="camera_to_lens_left" prefix="${prefix}" side="left"/>
   </xacro:macro>
 </robot>

File: aegis_description/urdf/modules/adapter_to_sensor.xacro (robot description, xacro)
@@ -40,16 +40,16 @@
     </joint>
     <link name="${prefix}adapter_to_sensor_end"/>
-    <joint name="${prefix}adapter_to_camera_mounting_back_joint" type="fixed">
+    <joint name="${prefix}adapter_to_mount_camera_tool_right_joint" type="fixed">
       <origin xyz="0 0 ${height_to_adapter}" rpy="0 ${pi} 0"/>
       <parent link="${prefix}adapter_to_sensor"/>
-      <child link="${prefix}adapter_to_camera_mounting_back"/>
+      <child link="${prefix}adapter_to_mount_camera_tool_right"/>
     </joint>
-    <link name="${prefix}adapter_to_camera_mounting_back"/>
-    <joint name="${prefix}adapter_to_camera_mounting_front_joint" type="fixed">
+    <link name="${prefix}adapter_to_mount_camera_tool_right"/>
+    <joint name="${prefix}adapter_to_mount_camera_tool_left_joint" type="fixed">
       <origin xyz="0 0 ${height_to_adapter}" rpy="0 ${pi} ${pi}"/>
       <parent link="${prefix}adapter_to_sensor"/>
-      <child link="${prefix}adapter_to_camera_mounting_front"/>
+      <child link="${prefix}adapter_to_mount_camera_tool_left"/>
     </joint>
-    <link name="${prefix}adapter_to_camera_mounting_front"/>
+    <link name="${prefix}adapter_to_mount_camera_tool_left"/>
   </xacro:macro>
 </robot>

File: aegis_description/urdf/modules/camera_tool_basler.xacro (robot description, xacro)
@@ -1,5 +1,5 @@
 <?xml version="1.0"?>
 <robot xmlns:xacro="http://ros.org/wiki/xacro">
-  <xacro:macro name="basler_camera" params="prefix parent side">
+  <xacro:macro name="camera_tool_basler" params="prefix parent side">
     <xacro:property name="camera_mass" value="0.217"/>
     <xacro:property name="camera_mounting_offset" value="0.0387"/>

File: aegis_description/urdf/modules/lens_computar.xacro (robot description, xacro)
@@ -2,14 +2,14 @@
 <robot xmlns:xacro="http://ros.org/wiki/xacro">
   <!-- <xacro:include filename="$(find aegis_description)/urdf/cylinders_inertial.xacro"/> -->
-  <xacro:macro name="computar_lens" params="prefix parent side">
+  <xacro:macro name="lens_computar" params="prefix parent side">
     <xacro:property name="lens_mass" value="0.063"/>
     <xacro:property name="lens_radius" value="0.01660"/>
     <xacro:property name="lens_height" value="0.02890"/>
-    <joint name="computar_lens_joint_${side}" type="fixed">
+    <joint name="lens_computar_joint_${side}" type="fixed">
       <origin xyz="0 0 0" rpy="0 0 0"/>
       <parent link="${parent}"/>
-      <child link="${prefix}computar_lens_${side}"/>
+      <child link="${prefix}lens_computar_${side}"/>
     </joint>
-    <link name="${prefix}computar_lens_${side}">
+    <link name="${prefix}lens_computar_${side}">
       <visual>
         <origin xyz="0 0 0" rpy="0 0 ${pi}"/>

File: aegis_description/urdf/modules/mount_camera_tool_basler.xacro (robot description, xacro)
@@ -1,5 +1,5 @@
 <?xml version="1.0"?>
 <robot xmlns:xacro="http://ros.org/wiki/xacro">
-  <xacro:macro name="basler_camera_mounting" params="prefix parent side">
+  <xacro:macro name="mount_camera_tool_balser" params="prefix parent side">
     <xacro:property name="mass" value="0.217"/>
     <xacro:property name="mounting_width" value="0.07000"/>
@@ -10,10 +10,10 @@
     <xacro:property name="mounting_dist_z" value="-0.06607"/>
     <xacro:property name="mounting_dist_x" value="0.119084"/>
-    <joint name="basler_camera_mounting_joint_${side}" type="fixed">
+    <joint name="mount_camera_tool_balser_joint_${side}" type="fixed">
       <origin xyz="0 0 0" rpy="0 0 0"/>
       <parent link="${parent}"/>
-      <child link="${prefix}basler_camera_mounting_${side}"/>
+      <child link="${prefix}mount_camera_tool_balser_${side}"/>
     </joint>
-    <link name="${prefix}basler_camera_mounting_${side}">
+    <link name="${prefix}mount_camera_tool_balser_${side}">
       <visual>
         <origin xyz="0 0 0" rpy="0 0 0"/>
@@ -30,10 +30,10 @@
       </collision>
     </link>
-    <joint name="${prefix}mounting_to_camera_${side}_joint" type="fixed">
+    <joint name="${prefix}mount_camera_tool_balser_${side}_joint" type="fixed">
       <origin xyz="${mounting_dist_x} 0 ${mounting_dist_z}" rpy="${mounting_yaw} 0 ${-0.5 * pi}"/>
-      <parent link="${prefix}basler_camera_mounting_${side}"/>
-      <child link="${prefix}mounting_to_camera_${side}"/>
+      <parent link="${prefix}mount_camera_tool_balser_${side}"/>
+      <child link="${prefix}mount_to_camera_${side}"/>
     </joint>
-    <link name="${prefix}mounting_to_camera_${side}"/>
+    <link name="${prefix}mount_to_camera_${side}"/>
   </xacro:macro>
 </robot>

Commit message: Change names and cameras collision

File: aegis_description/urdf/aegis.xacro (robot description, xacro)
@@ -20,13 +20,13 @@
     <xacro:adapter_from_sensor parent="tool_mount_link" prefix="${prefix}"/>
     <xacro:hande_gripper parent="adapter_from_sensor_end" prefix="${prefix}" mock_hardware="${mock_hardware}"/>
-    <xacro:mount_camera_tool_luxonis parent="mount" prefix="${prefix}"/>
-    <xacro:mount_camera_tool_balser parent="adapter_to_mount_camera_tool_right" prefix="${prefix}" side="right"/>
-    <xacro:mount_camera_tool_balser parent="adapter_to_mount_camera_tool_left" prefix="${prefix}" side="left"/>
+    <xacro:mount_camera_tool_luxonis parent="adapter_mount_front" prefix="${prefix}"/>
+    <xacro:mount_camera_tool_basler parent="adapter_mount_right" prefix="${prefix}" side="right"/>
+    <xacro:mount_camera_tool_basler parent="adapter_mount_left" prefix="${prefix}" side="left"/>
     <xacro:camera_scene_luxonis parent="cell"/>
-    <xacro:camera_tool_luxonis parent="camera_tool" prefix="${prefix}"/>
-    <xacro:camera_tool_basler parent="mount_to_camera_right" prefix="${prefix}" side="right"/>
-    <xacro:camera_tool_basler parent="mount_to_camera_left" prefix="${prefix}" side="left"/>
-    <xacro:lens_computar parent="camera_to_lens_right" prefix="${prefix}" side="right"/>
-    <xacro:lens_computar parent="camera_to_lens_left" prefix="${prefix}" side="left"/>
+    <xacro:camera_tool_luxonis parent="mount_front_end" prefix="${prefix}"/>
+    <xacro:camera_tool_basler parent="mount_right_end" prefix="${prefix}" side="right"/>
+    <xacro:camera_tool_basler parent="mount_left_end" prefix="${prefix}" side="left"/>
+    <xacro:lens_computar parent="cam_tool_right_basler" prefix="${prefix}" side="right"/>
+    <xacro:lens_computar parent="cam_tool_left_basler" prefix="${prefix}" side="left"/>
   </xacro:macro>
 </robot>

File: aegis_description/urdf/modules/adapter_to_sensor.xacro (robot description, xacro)
@@ -43,22 +43,22 @@
     </joint>
     <link name="${prefix}adapter_to_sensor_end"/>
-    <joint name="${prefix}adapter_to_mount_camera_tool_right_joint" type="fixed">
+    <joint name="${prefix}adapter_to_mount_right_joint" type="fixed">
       <origin xyz="0 0 ${height_to_adapter}" rpy="0 ${pi} 0"/>
       <parent link="${prefix}adapter_to_sensor"/>
-      <child link="${prefix}adapter_to_mount_camera_tool_right"/>
+      <child link="${prefix}adapter_mount_right"/>
     </joint>
-    <link name="${prefix}adapter_to_mount_camera_tool_right"/>
-    <joint name="${prefix}adapter_to_mount_camera_tool_left_joint" type="fixed">
+    <link name="${prefix}adapter_mount_right"/>
+    <joint name="${prefix}adapter_to_mount_left_joint" type="fixed">
       <origin xyz="0 0 ${height_to_adapter}" rpy="0 ${pi} ${pi}"/>
       <parent link="${prefix}adapter_to_sensor"/>
-      <child link="${prefix}adapter_to_mount_camera_tool_left"/>
+      <child link="${prefix}adapter_mount_left"/>
     </joint>
-    <link name="${prefix}adapter_to_mount_camera_tool_left"/>
-    <joint name="adapter_to_mount_joint" type="fixed">
+    <link name="${prefix}adapter_mount_left"/>
+    <joint name="${prefix}adapter_to_mount_front_joint" type="fixed">
       <origin xyz="0 0 ${height_to_adapter}" rpy="0 ${pi} ${pi / 2}"/>
       <parent link="${prefix}adapter_to_sensor"/>
-      <child link="${prefix}mount"/>
+      <child link="${prefix}adapter_mount_front"/>
     </joint>
-    <link name="${prefix}mount"/>
+    <link name="${prefix}adapter_mount_front"/>
   </xacro:macro>
 </robot>

File: aegis_description/urdf/modules/camera_tool_basler.xacro (robot description, xacro)
@@ -7,10 +7,10 @@
     <xacro:property name="camera_length" value="0.0603"/>
     <xacro:property name="lens_offset" value="-0.0145"/>
-    <joint name="basler_camera_joint_${side}" type="fixed">
+    <joint name="${prefix}camera_${side}_joint" type="fixed">
       <origin xyz="0 ${0.5 * camera_height} ${camera_mounting_offset}" rpy="0 0 0"/>
       <parent link="${parent}"/>
-      <child link="${prefix}basler_camera_${side}"/>
+      <child link="${prefix}cam_tool_${side}_basler"/>
     </joint>
-    <link name="${prefix}basler_camera_${side}">
+    <link name="${prefix}cam_tool_${side}_basler">
       <visual>
         <origin xyz="0 0 0" rpy="0 0 0"/>
@@ -24,17 +24,5 @@
         <inertia ixx="0.3403" ixy="0.0" ixz="0.0" iyy="0.3403" iyz="0.0" izz="0.039606138"/>
       </inertial>
-      <collision>
-        <origin xyz="0 0 ${0.5 * camera_length}" rpy="0 0 0"/>
-        <geometry>
-          <box size="${camera_height} ${camera_height} ${camera_length}"/>
-        </geometry>
-      </collision>
     </link>
-    <joint name="${prefix}camera_to_lens_${side}_joint" type="fixed">
-      <origin xyz="0 0 ${lens_offset}" rpy="0 0 0"/>
-      <parent link="${prefix}basler_camera_${side}"/>
-      <child link="${prefix}camera_to_lens_${side}"/>
-    </joint>
-    <link name="${prefix}camera_to_lens_${side}"/>
   </xacro:macro>
 </robot>

File: aegis_description/urdf/modules/lens_computar.xacro (robot description, xacro)
@@ -5,10 +5,11 @@
     <xacro:property name="lens_radius" value="0.01660"/>
     <xacro:property name="lens_height" value="0.02890"/>
-    <joint name="lens_computar_joint_${side}" type="fixed">
-      <origin xyz="0 0 0" rpy="0 0 0"/>
+    <xacro:property name="lens_offset" value="-0.0145"/>
+    <joint name="lens_${side}_joint" type="fixed">
+      <origin xyz="0 0 ${lens_offset}" rpy="0 0 0"/>
       <parent link="${parent}"/>
-      <child link="${prefix}lens_computar_${side}"/>
+      <child link="${prefix}lens_${side}_computar"/>
     </joint>
-    <link name="${prefix}lens_computar_${side}">
+    <link name="${prefix}lens_${side}_computar">
       <visual>
         <origin xyz="0 0 0" rpy="0 0 ${pi}"/>
@@ -32,10 +33,4 @@
         />
       </inertial>
-      <collision>
-        <origin xyz="0 0 0" rpy="0 0 ${pi}"/>
-        <geometry>
-          <cylinder radius="${lens_radius}" length="${lens_height}"/>
-        </geometry>
-      </collision>
     </link>
   </xacro:macro>

File: aegis_description/urdf/modules/mount_camera_tool_basler.xacro (robot description, xacro)
@@ -1,5 +1,5 @@
 <?xml version="1.0"?>
 <robot xmlns:xacro="http://ros.org/wiki/xacro">
-  <xacro:macro name="mount_camera_tool_balser" params="prefix parent side">
+  <xacro:macro name="mount_camera_tool_basler" params="prefix parent side">
     <xacro:property name="mass" value="0.217"/>
     <xacro:property name="mounting_width" value="0.07000"/>
@@ -10,10 +10,10 @@
     <xacro:property name="mounting_dist_z" value="-0.06607"/>
     <xacro:property name="mounting_dist_x" value="0.119084"/>
-    <joint name="mount_camera_tool_balser_joint_${side}" type="fixed">
+    <joint name="${prefix}mount_${side}_joint" type="fixed">
       <origin xyz="0 0 0" rpy="0 0 0"/>
       <parent link="${parent}"/>
-      <child link="${prefix}mount_camera_tool_balser_${side}"/>
+      <child link="${prefix}mount_${side}"/>
     </joint>
-    <link name="${prefix}mount_camera_tool_balser_${side}">
+    <link name="${prefix}mount_${side}">
       <visual>
         <origin xyz="0 0 0" rpy="0 0 0"/>
@@ -28,16 +28,40 @@
       </inertial>
       <collision>
-        <origin xyz="${1.0 * mounting_size_x} 0 ${-1.0 * mounting_height}" rpy="0 0 0"/>
+        <origin xyz="0.048 0 0" rpy="0 0 0"/>
         <geometry>
-          <box size="${mounting_size_x} ${mounting_width} ${3.0 * mounting_height}"/>
+          <box size="0.01 0.086 0.06"/>
+        </geometry>
+      </collision>
+      <collision>
+        <origin xyz="0.11 0 -0.026" rpy="0 0 0"/>
+        <geometry>
+          <box size="0.114 0.04 0.088"/>
+        </geometry>
+      </collision>
+      <collision>
+        <origin xyz="0.105 0 -0.08" rpy="0 0 0"/>
+        <geometry>
+          <box size="0.104 0.04 0.02"/>
+        </geometry>
+      </collision>
+      <collision>
+        <origin xyz="0.096 0 -0.1" rpy="0 0 0"/>
+        <geometry>
+          <box size="0.086 0.04 0.02"/>
+        </geometry>
+      </collision>
+      <collision>
+        <origin xyz="0.091 0 -0.125" rpy="0 0 0"/>
+        <geometry>
+          <box size="0.076 0.04 0.03"/>
         </geometry>
       </collision>
     </link>
-    <joint name="${prefix}mount_camera_tool_balser_${side}_joint" type="fixed">
+    <joint name="${prefix}mount_${side}_end_joint" type="fixed">
       <origin xyz="${mounting_dist_x} 0 ${mounting_dist_z}" rpy="${mounting_yaw} 0 ${-0.5 * pi}"/>
-      <parent link="${prefix}mount_camera_tool_balser_${side}"/>
-      <child link="${prefix}mount_to_camera_${side}"/>
+      <parent link="${prefix}mount_${side}"/>
+      <child link="${prefix}mount_${side}_end"/>
     </joint>
-    <link name="${prefix}mount_to_camera_${side}"/>
+    <link name="${prefix}mount_${side}_end"/>
   </xacro:macro>
 </robot>

File: aegis_description/urdf/modules/mount_camera_tool_luxonis.xacro (robot description, xacro)
@@ -3,12 +3,10 @@
   <xacro:macro name="mount_camera_tool_luxonis" params="prefix parent">
     <xacro:property name="mass" value="0.4"/>
-    <xacro:property name="mounting_dist_x" value="0.091"/>
-    <xacro:property name="mounting_dist_z" value="-0.014"/>
-    <joint name="${prefix}mount_camera_joint" type="fixed">
+    <joint name="${prefix}mount_front_joint" type="fixed">
       <origin xyz="0 0 0" rpy="0 0 0"/>
       <parent link="${parent}"/>
-      <child link="${prefix}mount_camera"/>
+      <child link="${prefix}mount_front"/>
     </joint>
-    <link name="${prefix}mount_camera">
+    <link name="${prefix}mount_front">
       <visual>
         <origin xyz="0 0 0" rpy="0 0 0"/>
@@ -23,16 +21,16 @@
       </inertial>
       <collision>
-        <origin xyz="0.084 0 -0.01" rpy="0 0 0"/>
+        <origin xyz="0.084 0 0" rpy="0 0 0"/>
         <geometry>
-          <box size="0.076 0.1 0.12"/>
+          <box size="0.08 0.1 0.142"/>
         </geometry>
       </collision>
     </link>
-    <joint name="${prefix}mount_to_camera_joint" type="fixed">
+    <joint name="${prefix}mount_front_end_joint" type="fixed">
       <origin xyz="0.091 0 -0.012" rpy="0 0 ${-pi}"/>
-      <parent link="${prefix}mount_camera"/>
-      <child link="${prefix}camera_tool"/>
+      <parent link="${prefix}mount_front"/>
+      <child link="${prefix}mount_front_end"/>
     </joint>
-    <link name="${prefix}camera_tool"/>
+    <link name="${prefix}mount_front_end"/>
   </xacro:macro>
 </robot>

Commit message: Change names

File: aegis_description/urdf/aegis.xacro (robot description, xacro)
@@ -27,6 +27,6 @@
     <xacro:camera_tool_basler parent="mount_right_end" prefix="${prefix}" side="right"/>
     <xacro:camera_tool_basler parent="mount_left_end" prefix="${prefix}" side="left"/>
-    <xacro:lens_computar parent="cam_tool_right_basler" prefix="${prefix}" side="right"/>
-    <xacro:lens_computar parent="cam_tool_left_basler" prefix="${prefix}" side="left"/>
+    <xacro:lens_computar parent="cam_tool_right" prefix="${prefix}" side="right"/>
+    <xacro:lens_computar parent="cam_tool_left" prefix="${prefix}" side="left"/>
   </xacro:macro>
 </robot>

File: aegis_description/urdf/modules/camera_tool_basler.xacro (robot description, xacro)
@@ -10,7 +10,7 @@
       <origin xyz="0 ${0.5 * camera_height} ${camera_mounting_offset}" rpy="0 0 0"/>
       <parent link="${parent}"/>
-      <child link="${prefix}cam_tool_${side}_basler"/>
+      <child link="${prefix}cam_tool_${side}"/>
     </joint>
-    <link name="${prefix}cam_tool_${side}_basler">
+    <link name="${prefix}cam_tool_${side}">
       <visual>
         <origin xyz="0 0 0" rpy="0 0 0"/>

File: aegis_description/urdf/modules/lens_computar.xacro (robot description, xacro)
@@ -9,7 +9,7 @@
       <origin xyz="0 0 ${lens_offset}" rpy="0 0 0"/>
       <parent link="${parent}"/>
-      <child link="${prefix}lens_${side}_computar"/>
+      <child link="${prefix}lens_${side}"/>
     </joint>
-    <link name="${prefix}lens_${side}_computar">
+    <link name="${prefix}lens_${side}">
       <visual>
         <origin xyz="0 0 0" rpy="0 0 ${pi}"/>

Commit message: CHG: moved ur_base to world

File: aegis_description/urdf/aegis.xacro (robot description, xacro)
@@ -14,6 +14,6 @@
   <xacro:include filename="$(find aegis_description)/urdf/modules/lens_computar.xacro"/>
   <xacro:macro name="aegis_robot" params="parent tf_prefix prefix mock_hardware">
-    <xacro:cell parent="${parent}"/>
-    <xacro:ur_definition name="aegis" parent="ur_base" tf_prefix="${tf_prefix}" mock_hardware="${mock_hardware}"/>
+    <xacro:ur_definition name="aegis" parent="${parent}" tf_prefix="${tf_prefix}" mock_hardware="${mock_hardware}"/>
+    <xacro:cell parent="ur_base"/>
     <xacro:adapter_to_sensor parent="tool0" prefix="${prefix}"/>
     <xacro:ft_sensor_schunk_axia80 parent="adapter_to_sensor_end" prefix="${prefix}" mock_hardware="${mock_hardware}"/>

File: aegis_description/urdf/modules/cell.xacro (robot description, xacro)
@@ -2,7 +2,7 @@
 <robot xmlns:xacro="http://ros.org/wiki/xacro">
   <xacro:macro name="cell" params="parent">
-    <joint name="world_to_cell_joint" type="fixed">
-      <origin xyz="0 0 0" rpy="0 0 0"/>
-      <parent link="${parent}"/>
+    <joint name="ur_base_to_cell" type="fixed">
+      <origin xyz="0 0 -0.806" rpy="0 0 -${0.5 * pi}"/>
+      <parent link="ur_base"/>
       <child link="cell"/>
     </joint>
@@ -63,9 +63,4 @@
       </collision>
     </link>
-    <joint name="cell_to_ur_base" type="fixed">
-      <origin xyz="0 0 0.806" rpy="0 0 ${0.5 * pi}"/>
-      <parent link="cell"/>
-      <child link="ur_base"/>
-    </joint>
     <link name="ur_base"/>
   </xacro:macro>

File: aegis_description/urdf/modules/ur_definition.xacro (robot description, xacro)
@@ -2,4 +2,10 @@
 <robot xmlns:xacro="http://ros.org/wiki/xacro">
   <xacro:include filename="$(find ur_description)/urdf/ur_macro.xacro"/>
+  <!-- For simulation, the global parent must be the same as ur_base -->
+  <joint name="world_to_ur_base" type="fixed">
+    <origin xyz="0 0 0" rpy="0 0 0"/>
+    <parent link="${parent}"/>
+    <child link="ur_base"/>
+  </joint>
   <!-- The list of all available options can be found in the <ur_description>/urdf/ur_macro.xacro file -->
   <!-- Descriptions of the arguments can be found in the <ur_robot_driver>/src/hardware_interface.cpp file -->
@@ -40,5 +46,5 @@
       name="${name}"
       tf_prefix="$(arg tf_prefix)"
-      parent="${parent}"
+      parent="ur_base"
       joint_limits_parameters_file="$(arg joint_limit_params)"
       kinematics_parameters_file="$(arg kinematics_calibration)"
@@ -68,5 +74,5 @@
     <xacro:if value="$(arg sim_gazebo)">
       <!-- Gazebo plugins -->
-      <gazebo reference="${parent}"/>
+      <gazebo reference="ur_base"/>
       <gazebo>
         <plugin filename="libgazebo_ros2_control.so" name="gazebo_ros2_control">
@@ -77,5 +83,5 @@
     <xacro:if value="$(arg sim_ignition)">
       <!-- Gazebo plugins -->
-      <gazebo reference="${parent}"/>
+      <gazebo reference="ur_base"/>
       <gazebo>
         <plugin filename="libign_ros2_control-system.so" name="ign_ros2_control::IgnitionROS2ControlPlugin">
