Commit message: CHG: cleanup

File: aegis_description/urdf/aegis.xacro (robot description, xacro)
@@ -14,6 +14,6 @@
   <xacro:include filename="$(find aegis_description)/urdf/modules/lens_computar.xacro"/>
   <xacro:macro name="aegis_robot" params="parent tf_prefix prefix mock_hardware">
+    <xacro:cell parent="${parent}"/>
     <xacro:ur_definition name="aegis" parent="${parent}" tf_prefix="${tf_prefix}" mock_hardware="${mock_hardware}"/>
-    <xacro:cell parent="${parent}"/>
     <xacro:adapter_to_sensor parent="tool0" prefix="${prefix}"/>
     <xacro:ft_sensor_schunk_axia80 parent="adapter_to_sensor_end" prefix="${prefix}" mock_hardware="${mock_hardware}"/>

File: aegis_description/urdf/modules/cell.xacro (robot description, xacro)
@@ -2,5 +2,5 @@
 <robot xmlns:xacro="http://ros.org/wiki/xacro">
   <xacro:macro name="cell" params="parent">
-    <joint name="ur_base_to_cell" type="fixed">
+    <joint name="parent_to_cell" type="fixed">
       <origin xyz="0 0 -0.806" rpy="0 0 -${0.5 * pi}"/>
       <parent link="${parent}"/>

File: aegis_description/urdf/modules/ur_definition.xacro (robot description, xacro)
@@ -68,5 +68,5 @@
     <xacro:if value="$(arg sim_gazebo)">
       <!-- Gazebo plugins -->
-      <gazebo reference="ur_base"/>
+      <gazebo reference="${parent}"/>
       <gazebo>
         <plugin filename="libgazebo_ros2_control.so" name="gazebo_ros2_control">
@@ -77,5 +77,5 @@
     <xacro:if value="$(arg sim_ignition)">
       <!-- Gazebo plugins -->
-      <gazebo reference="ur_base"/>
+      <gazebo reference="${parent}"/>
       <gazebo>
         <plugin filename="libign_ros2_control-system.so" name="ign_ros2_control::IgnitionROS2ControlPlugin">

Commit message: Move cell disabling logic

File: aegis_description/urdf/aegis.xacro (robot description, xacro)
@@ -14,7 +14,5 @@
   <xacro:include filename="$(find aegis_description)/urdf/modules/lens_computar.xacro"/>
   <xacro:macro name="aegis_robot" params="parent tf_prefix prefix mock_hardware disable_cell disable_cell_collision">
-    <xacro:unless value="${disable_cell}">
-      <xacro:cell parent="${parent}" disable_cell_collision="${disable_cell_collision}"/>
-    </xacro:unless>
+    <xacro:cell parent="${parent}" disable_cell="${disable_cell}" disable_cell_collision="${disable_cell_collision}"/>
     <xacro:ur_definition name="aegis" parent="${parent}" tf_prefix="${tf_prefix}" mock_hardware="${mock_hardware}"/>
     <xacro:adapter_to_sensor parent="tool0" prefix="${prefix}"/>

File: aegis_description/urdf/modules/cell.xacro (robot description, xacro)
@@ -1,68 +1,70 @@
 <?xml version="1.0"?>
 <robot xmlns:xacro="http://ros.org/wiki/xacro">
-  <xacro:macro name="cell" params="parent disable_cell_collision">
-    <joint name="world_to_cell" type="fixed">
-      <origin xyz="0 0 -0.806" rpy="0 0 -${0.5 * pi}"/>
-      <parent link="${parent}"/>
-      <child link="cell"/>
-    </joint>
-    <link name="cell">
-      <visual>
-        <origin xyz="-0.460 -0.240 0.786" rpy="0 0 0"/>
-        <geometry>
-          <mesh filename="package://aegis_description/meshes/cell.dae" scale="1.0 1.0 1.0"/>
-        </geometry>
-      </visual>
-      <xacro:unless value="${disable_cell_collision}">
-        <collision>
-          <origin xyz="0 -0.162 0.435" rpy="0 0 0"/>
+  <xacro:macro name="cell" params="parent disable_cell disable_cell_collision">
+    <xacro:unless value="${disable_cell}">
+      <joint name="world_to_cell" type="fixed">
+        <origin xyz="0 0 -0.806" rpy="0 0 -${0.5 * pi}"/>
+        <parent link="${parent}"/>
+        <child link="cell"/>
+      </joint>
+      <link name="cell">
+        <visual>
+          <origin xyz="-0.460 -0.240 0.786" rpy="0 0 0"/>
           <geometry>
-            <box size="0.72 0.324 0.87"/>
+            <mesh filename="package://aegis_description/meshes/cell.dae" scale="1.0 1.0 1.0"/>
           </geometry>
-        </collision>
-        <collision>
-          <origin xyz="0 0.162 0.41" rpy="0 0 0"/>
-          <geometry>
-            <box size="0.72 0.324 0.82"/>
-          </geometry>
-        </collision>
-        <collision>
-          <origin xyz="0.48 0 0.97" rpy="0 0 0"/>
-          <geometry>
-            <box size="0.08 0.648 1.94"/>
-          </geometry>
-        </collision>
-        <collision>
-          <origin xyz="0.4 0 0.435" rpy="0 0 0"/>
-          <geometry>
-            <box size="0.08 0.648 0.87"/>
-          </geometry>
-        </collision>
-        <collision>
-          <origin xyz="-0.48 0 0.97" rpy="0 0 0"/>
-          <geometry>
-            <box size="0.08 0.648 1.94"/>
-          </geometry>
-        </collision>
-        <collision>
-          <origin xyz="-0.4 0 0.435" rpy="0 0 0"/>
-          <geometry>
-            <box size="0.08 0.648 0.87"/>
-          </geometry>
-        </collision>
-        <collision>
-          <origin xyz="0 0.04 1.98" rpy="0 0 0"/>
-          <geometry>
-            <box size="1.04 0.728 0.08"/>
-          </geometry>
-        </collision>
-        <collision>
-          <origin xyz="0 -0.62 1.2" rpy="0 0 0"/>
-          <geometry>
-            <box size="2.4 0.02 2.4"/>
-          </geometry>
-        </collision>
-      </xacro:unless>
-    </link>
+        </visual>
+        <xacro:unless value="${disable_cell_collision}">
+          <collision>
+            <origin xyz="0 -0.162 0.435" rpy="0 0 0"/>
+            <geometry>
+              <box size="0.72 0.324 0.87"/>
+            </geometry>
+          </collision>
+          <collision>
+            <origin xyz="0 0.162 0.41" rpy="0 0 0"/>
+            <geometry>
+              <box size="0.72 0.324 0.82"/>
+            </geometry>
+          </collision>
+          <collision>
+            <origin xyz="0.48 0 0.97" rpy="0 0 0"/>
+            <geometry>
+              <box size="0.08 0.648 1.94"/>
+            </geometry>
+          </collision>
+          <collision>
+            <origin xyz="0.4 0 0.435" rpy="0 0 0"/>
+            <geometry>
+              <box size="0.08 0.648 0.87"/>
+            </geometry>
+          </collision>
+          <collision>
+            <origin xyz="-0.48 0 0.97" rpy="0 0 0"/>
+            <geometry>
+              <box size="0.08 0.648 1.94"/>
+            </geometry>
+          </collision>
+          <collision>
+            <origin xyz="-0.4 0 0.435" rpy="0 0 0"/>
+            <geometry>
+              <box size="0.08 0.648 0.87"/>
+            </geometry>
+          </collision>
+          <collision>
+            <origin xyz="0 0.04 1.98" rpy="0 0 0"/>
+            <geometry>
+              <box size="1.04 0.728 0.08"/>
+            </geometry>
+          </collision>
+          <collision>
+            <origin xyz="0 -0.62 1.2" rpy="0 0 0"/>
+            <geometry>
+              <box size="2.4 0.02 2.4"/>
+            </geometry>
+          </collision>
+        </xacro:unless>
+      </link>
+    </xacro:unless>
   </xacro:macro>
 </robot>
