Commit message: names changed, added parameter for wled suporters, moved definitions to cell.xacro

File: aegis_description/urdf/aegis.xacro (robot description, xacro)
@@ -2,6 +2,6 @@
 <robot xmlns:xacro="http://wiki.ros.org/xacro">
   <xacro:include filename="$(find aegis_description)/urdf/modules/cell.xacro"/>
-  <xacro:include filename="$(find aegis_description)/urdf/modules/wled_lights_right.xacro" />
-  <xacro:include filename="$(find aegis_description)/urdf/modules/wled_lights_left.xacro" />
+  <xacro:include filename="$(find aegis_description)/urdf/modules/light_support_right.xacro" />
+  <xacro:include filename="$(find aegis_description)/urdf/modules/light_support_left.xacro" />
   <xacro:include filename="$(find aegis_description)/urdf/modules/adapter_cell.xacro"/>
   <xacro:include filename="$(find aegis_description)/urdf/modules/ur_definition.xacro"/>
@@ -16,9 +16,7 @@
   <xacro:include filename="$(find aegis_description)/urdf/modules/camera_tool_basler.xacro"/>
   <xacro:include filename="$(find aegis_description)/urdf/modules/lens_computar.xacro"/>
-  <xacro:macro name="aegis_robot" params="parent tf_prefix prefix mock_hardware disable_cell disable_cell_collision">
-    <xacro:cell parent="${parent}" disable_cell="${disable_cell}" disable_cell_collision="${disable_cell_collision}"/>
-    <xacro:wled_lights_right parent="${parent}" prefix="${prefix}"/>
-    <xacro:wled_lights_left parent="${parent}" prefix="${prefix}"/>
-    <xacro:adapter_cell parent="${parent}" prefix="${prefix}" disable_cell="${disable_cell}" disable_cell_collision="${disable_cell_collision}"/>
+  <xacro:macro name="aegis_robot" params="parent tf_prefix prefix mock_hardware disable_cell disable_cell_collision disable_leds:=false">
+    <xacro:cell parent="${parent}" disable_cell="${disable_cell}" disable_cell_collision="${disable_cell_collision}" disable_leds="${disable_leds}"/>
+    <xacro:adapter_cell parent="${parent}" prefix="${prefix}" disable_cell="${disable_cell}" disable_cell_collision="${disable_cell_collision}" disable_leds="${disable_leds}"/>
     <xacro:ur_definition name="aegis" parent="${parent}" tf_prefix="${tf_prefix}" mock_hardware="${mock_hardware}"/>
     <xacro:adapter_to_sensor parent="tool0" prefix="${prefix}"/>

File: aegis_description/urdf/modules/cell.xacro (robot description, xacro)
@@ -66,4 +66,6 @@
         </xacro:unless>
       </link>
+      <xacro:wled_lights_right parent="cell" prefix=""/>
+      <xacro:wled_lights_left parent="cell" prefix=""/>
     </xacro:unless>
   </xacro:macro>

Commit message: all fixes

File: aegis_description/urdf/aegis.xacro (robot description, xacro)
@@ -2,6 +2,6 @@
 <robot xmlns:xacro="http://wiki.ros.org/xacro">
   <xacro:include filename="$(find aegis_description)/urdf/modules/cell.xacro"/>
-  <xacro:include filename="$(find aegis_description)/urdf/modules/light_support_right.xacro" />
-  <xacro:include filename="$(find aegis_description)/urdf/modules/light_support_left.xacro" />
+  <xacro:include filename="$(find aegis_description)/urdf/modules/lighting_support_right.xacro" />
+  <xacro:include filename="$(find aegis_description)/urdf/modules/lighting_support_left.xacro" />
   <xacro:include filename="$(find aegis_description)/urdf/modules/adapter_cell.xacro"/>
   <xacro:include filename="$(find aegis_description)/urdf/modules/ur_definition.xacro"/>
@@ -16,5 +16,5 @@
   <xacro:include filename="$(find aegis_description)/urdf/modules/camera_tool_basler.xacro"/>
   <xacro:include filename="$(find aegis_description)/urdf/modules/lens_computar.xacro"/>
-  <xacro:macro name="aegis_robot" params="parent tf_prefix prefix mock_hardware disable_cell disable_cell_collision disable_leds:=false">
+  <xacro:macro name="aegis_robot" params="parent tf_prefix prefix mock_hardware disable_cell disable_cell_collision disable_leds">
     <xacro:cell parent="${parent}" disable_cell="${disable_cell}" disable_cell_collision="${disable_cell_collision}" disable_leds="${disable_leds}"/>
     <xacro:adapter_cell parent="${parent}" prefix="${prefix}" disable_cell="${disable_cell}" disable_cell_collision="${disable_cell_collision}"/>

File: aegis_description/urdf/modules/lighting_support_left.xacro (robot description, xacro)
@@ -1,15 +1,15 @@
 <?xml version="1.0"?>
 <robot xmlns:xacro="http://ros.org/wiki/xacro">
-  <xacro:macro name="wled_lights_right" params="parent prefix">
-    <joint name="${prefix}wled_lights_right_joint" type="fixed">
-      <origin xyz="0.32 0.50 0.35" rpy="0.0 0.0 ${pi}"/>
+  <xacro:macro name="lighting_support_left" params="parent prefix">
+    <joint name="${prefix}lighting_support_left_joint" type="fixed">
+      <origin xyz="0.32 0.495 0.35" rpy="0.0 0.0 ${pi}"/>
       <parent link="${parent}"/>
-      <child link="${prefix}wled_lights_right_link"/>
+      <child link="${prefix}lighting_support_left_link"/>
     </joint>
-    <link name="${prefix}wled_lights_right_link">
+    <link name="${prefix}lighting_support_left_link">
       <visual>
         <origin xyz="0 0 0" rpy="0 0 0"/>
         <geometry>
-          <mesh filename="package://aegis_description/meshes/wled_lights_right.dae" scale="0.001 0.001 0.001"/>
+          <mesh filename="package://aegis_description/meshes/lighting_support_left.dae" scale="0.001 0.001 0.001"/>
         </geometry>
       </visual>
@@ -17,5 +17,5 @@
         <origin xyz="0 0 0" rpy="0 0 0"/>
         <geometry>
-          <mesh filename="package://aegis_description/meshes/wled_lights_right.dae" scale="0.001 0.001 0.001"/>
+          <mesh filename="package://aegis_description/meshes/lighting_support_left.dae" scale="0.001 0.001 0.001"/>
         </geometry>
       </collision>

File: aegis_description/urdf/modules/lighting_support_right.xacro (robot description, xacro)
@@ -1,15 +1,15 @@
 <?xml version="1.0"?>
 <robot xmlns:xacro="http://ros.org/wiki/xacro">
-  <xacro:macro name="wled_lights_left" params="parent prefix">
-    <joint name="${prefix}wled_lights_left_joint" type="fixed">
-      <origin xyz="0.32 0.495 0.35" rpy="0.0 0.0 ${pi}"/>
+  <xacro:macro name="lighting_support_right" params="parent prefix">
+    <joint name="${prefix}lighting_support_right_joint" type="fixed">
+      <origin xyz="0.32 0.50 0.35" rpy="0.0 0.0 ${pi}"/>
       <parent link="${parent}"/>
-      <child link="${prefix}wled_lights_left_link"/>
+      <child link="${prefix}lighting_support_right_link"/>
     </joint>
-    <link name="${prefix}wled_lights_left_link">
+    <link name="${prefix}lighting_support_right_link">
       <visual>
         <origin xyz="0 0 0" rpy="0 0 0"/>
         <geometry>
-          <mesh filename="package://aegis_description/meshes/wled_lights_left.dae" scale="0.001 0.001 0.001"/>
+          <mesh filename="package://aegis_description/meshes/lighting_support_right.dae" scale="0.001 0.001 0.001"/>
         </geometry>
       </visual>
@@ -17,5 +17,5 @@
         <origin xyz="0 0 0" rpy="0 0 0"/>
         <geometry>
-          <mesh filename="package://aegis_description/meshes/wled_lights_left.dae" scale="0.001 0.001 0.001"/>
+          <mesh filename="package://aegis_description/meshes/lighting_support_right.dae" scale="0.001 0.001 0.001"/>
         </geometry>
       </collision>
