Commit message: merged ceai_ur_moveit_config

File: aegis_moveit_config/urdf/aegis.ros2_control.xacro (robot description, xacro)
@@ -2,5 +2,5 @@
 <robot xmlns:xacro="http://www.ros.org/wiki/xacro">
   <xacro:macro name="aegis_ros2_control" params="name initial_positions_file">
-    <xacro:property name="initial_positions" value="${load_yaml(initial_positions_file)['initial_positions']}"/>
+    <xacro:property name="initial_positions" value="${xacro.load_yaml(initial_positions_file)['initial_positions']}"/>
     <ros2_control name="${name}" type="system">
       <hardware>

File: aegis_moveit_config/urdf/aegis.urdf.xacro (robot description, xacro)
@@ -3,5 +3,5 @@
   <xacro:arg name="initial_positions_file" default="initial_positions.yaml"/>
   <!-- Import aegis urdf file -->
-  <xacro:include filename="$(find aegis_description)/urdf/aegis.urdf.xacro"/>
+  <xacro:include filename="$(find ceai_ur_description)/urdf/aegis.urdf.xacro"/>
   <!-- Import control_xacro -->
   <xacro:include filename="aegis.ros2_control.xacro"/>
