Commit message: wip on debugging

File: aegis_control/urdf/aegis.ros2_control.xacro (robot description, xacro)
@@ -1,5 +1,5 @@
 <?xml version="1.0"?>
 <robot xmlns:xacro="http://www.ros.org/wiki/xacro">
-  <xacro:macro name="aegis_ros2_control" params="use_mock_hardware mock_sensor_commands">
+  <xacro:macro name="aegis_ros2_control" params="mock_hardware">
     <xacro:property name="initial_positions" value="${xacro.load_yaml(initial_positions_file)['initial_positions']}"/>
     <ros2_control name="${name}" type="system">

File: aegis_control/urdf/aegis_control.urdf.xacro (robot description, xacro)
@@ -1,10 +1,11 @@
 <?xml version="1.0"?>
 <robot xmlns:xacro="http://www.ros.org/wiki/xacro" name="aegis">
-  <xacro:arg name="use_mock_hardware" default="false"/>
-  <xacro:arg name="mock_sensor_commands" default="false"/>
+  <xacro:arg name="base_link" default="ur_base"/>
+  <xacro:arg name="prefix" default=""/>
+  <xacro:arg name="mock_hardware" default="false"/>
   <xacro:include filename="$(find aegis_description)/urdf/aegis.xacro"/>
   <xacro:include filename="$(find aegis_control)/urdf/aegis.ros2_control.xacro"/>
-  <link name="ur_base"/>
-  <xacro:aegis_robot parent="ur_base" prefix=""/>
-  <xacro:aegis_ros2_control use_mock_hardware="$(arg use_mock_hardware)" mock_sensor_commands="$(arg mock_sensor_commands)"/>
+  <link name="$(arg base_link)"/>
+  <xacro:aegis_robot parent="$(arg base_link)" prefix="$(arg prefix)" kinematics_calibration="$(find aegis_control)/config/ur_calibration.yaml" mock_hardware="$(arg mock_hardware)"/>
+  <xacro:aegis_ros2_control mock_hardware="$(arg mock_hardware)"/>
 </robot>

File: aegis_description/urdf/aegis.xacro (robot description, xacro)
@@ -5,11 +5,11 @@
   <xacro:include filename="$(find aegis_description)/urdf/modules/ft_schunk_axia80.xacro"/>
   <xacro:include filename="$(find aegis_description)/urdf/modules/adapter_from_sensor.xacro"/>
-  <xacro:include filename="$(find robotiq_hande_description)/urdf/modules/robotiq_hande_gripper.xacro"/>
-  <xacro:macro name="aegis_robot" params="name parent prefix">
-    <xacro:ur_definition name="$(arg name)" parent="$(arg parent)" prefix=""/>
-    <xacro:adapter_to_sensor parent="tool0" prefix=""/>
-    <xacro:ft_sensor_schunk_axia80 parent="adapter_to_sensor_end" prefix=""/>
-    <xacro:adapter_from_sensor parent="tool_mount_link" prefix=""/>
-    <xacro:robotiq_hande_gripper parent="adapter_from_sensor_end" prefix=""/>
+  <xacro:include filename="$(find robotiq_hande_description)/urdf/robotiq_hande_gripper.xacro"/>
+  <xacro:macro name="aegis_robot" params="parent prefix kinematics_calibration mock_hardware">
+    <xacro:ur_definition name="aegis" parent="${parent}" prefix="${prefix}" kinematics_calibration="${kinematics_calibration}" fake_hardware="${mock_hardware}"/>
+    <xacro:adapter_to_sensor parent="tool0" prefix="${prefix}"/>
+    <xacro:ft_sensor_schunk_axia80 parent="adapter_to_sensor_end" prefix="${prefix}"/>
+    <xacro:adapter_from_sensor parent="tool_mount_link" prefix="${prefix}"/>
+    <xacro:robotiq_hande_gripper parent="adapter_from_sensor_end" prefix="${prefix}"/>
   </xacro:macro>
 </robot>

File: aegis_description/urdf/modules/ur_definition.xacro (robot description, xacro)
@@ -2,5 +2,5 @@
 <robot xmlns:xacro="http://ros.org/wiki/xacro">
   <xacro:include filename="$(find ur_description)/urdf/ur_macro.xacro"/>
-  <xacro:macro name="ur_definition" params="name kinematics_params fake_hardware">
+  <xacro:macro name="ur_definition" params="name parent prefix kinematics_calibration fake_hardware">
     <!-- possible 'ur_type' values: ur3, ur3e, ur5, ur5e, ur10, ur10e, ur16e, ur20 -->
     <!-- the default value should raise an error in case this was called without defining the
@@ -8,6 +8,6 @@
     <xacro:arg name="ur_type" default="ur5e"/>
     <!-- parameters -->
-    <xacro:arg name="tf_prefix" default=""/>
-    <!-- TODO(issue#1): It must be updated with real hardware paramas! -->
+    <xacro:arg name="tf_prefix" default="${prefix}"/>
+    <!-- TODO: It must be updated with real hardware paramas! -->
     <xacro:arg name="joint_limit_params" default="$(find ur_description)/config/$(arg ur_type)/joint_limits.yaml"/>
     <xacro:arg name="physical_params" default="$(find ur_description)/config/$(arg ur_type)/physical_parameters.yaml"/>
@@ -39,6 +39,6 @@
     <xacro:arg name="tool_tcp_port" default="54321"/>
     <!-- Simulation parameters -->
-    <xacro:arg name="use_fake_hardware" default="$(arg fake_hardware)"/>
-    <xacro:arg name="fake_sensor_commands" default="$(arg fake_hardware)"/>
+    <xacro:arg name="use_fake_hardware" default="${fake_hardware}"/>
+    <xacro:arg name="fake_sensor_commands" default="false"/>
     <xacro:arg name="sim_gazebo" default="false"/>
     <xacro:arg name="sim_ignition" default="false"/>
@@ -51,9 +51,9 @@
     <!-- arm -->
     <xacro:ur_robot
-      name="aegis"
+      name="${name}"
       tf_prefix="$(arg tf_prefix)"
-      parent="ur_base"
+      parent="${parent}"
       joint_limits_parameters_file="$(arg joint_limit_params)"
-      kinematics_parameters_file="$(arg kinematics_params)"
+      kinematics_parameters_file="${kinematics_calibration}"
       physical_parameters_file="$(arg physical_params)"
       visual_parameters_file="$(arg visual_params)"

Commit message: debugging xarco urdf files

File: aegis_control/urdf/aegis.ros2_control.xacro (robot description, xacro)
@@ -1,7 +1,7 @@
 <?xml version="1.0"?>
 <robot xmlns:xacro="http://www.ros.org/wiki/xacro">
-  <xacro:macro name="aegis_ros2_control" params="mock_hardware">
+  <xacro:macro name="aegis_ros2_control" params="initial_positions_file mock_hardware">
     <xacro:property name="initial_positions" value="${xacro.load_yaml(initial_positions_file)['initial_positions']}"/>
-    <ros2_control name="${name}" type="system">
+    <ros2_control name="aegis" type="system">
       <hardware>
         <!-- By default, set up controllers for simulation. This won't work on real hardware -->

File: aegis_control/urdf/aegis_control.urdf.xacro (robot description, xacro)
@@ -1,11 +1,12 @@
 <?xml version="1.0"?>
 <robot xmlns:xacro="http://www.ros.org/wiki/xacro" name="aegis">
+  <xacro:arg name="mock_hardware" default="false"/>
   <xacro:arg name="base_link" default="ur_base"/>
   <xacro:arg name="prefix" default=""/>
-  <xacro:arg name="mock_hardware" default="false"/>
+  <xacro:arg name="initial_positions_file" default="$(find aegis_control)/config/initial_positions.yaml"/>
   <xacro:include filename="$(find aegis_description)/urdf/aegis.xacro"/>
   <xacro:include filename="$(find aegis_control)/urdf/aegis.ros2_control.xacro"/>
   <link name="$(arg base_link)"/>
   <xacro:aegis_robot parent="$(arg base_link)" prefix="$(arg prefix)" kinematics_calibration="$(find aegis_control)/config/ur_calibration.yaml" mock_hardware="$(arg mock_hardware)"/>
-  <xacro:aegis_ros2_control mock_hardware="$(arg mock_hardware)"/>
+  <xacro:aegis_ros2_control initial_positions_file="$(arg initial_positions_file)" mock_hardware="$(arg mock_hardware)"/>
 </robot>

File: aegis_description/urdf/aegis.xacro (robot description, xacro)
@@ -7,7 +7,7 @@
   <xacro:include filename="$(find robotiq_hande_description)/urdf/robotiq_hande_gripper.xacro"/>
   <xacro:macro name="aegis_robot" params="parent prefix kinematics_calibration mock_hardware">
-    <xacro:ur_definition name="aegis" parent="${parent}" prefix="${prefix}" kinematics_calibration="${kinematics_calibration}" fake_hardware="${mock_hardware}"/>
+    <xacro:ur_definition name="aegis" parent="${parent}" prefix="${prefix}" kinematics_calibration="${kinematics_calibration}" mock_hardware="${mock_hardware}"/>
     <xacro:adapter_to_sensor parent="tool0" prefix="${prefix}"/>
-    <xacro:ft_sensor_schunk_axia80 parent="adapter_to_sensor_end" prefix="${prefix}"/>
+    <xacro:ft_sensor_schunk_axia80 parent="adapter_to_sensor_end" prefix="${prefix}" mock_hardware="${mock_hardware}"/>
     <xacro:adapter_from_sensor parent="tool_mount_link" prefix="${prefix}"/>
     <xacro:robotiq_hande_gripper parent="adapter_from_sensor_end" prefix="${prefix}"/>

File: aegis_description/urdf/modules/ft_schunk_axia80.xacro (robot description, xacro)
@@ -12,10 +12,9 @@
   <xacro:arg name="use_hardware_biasing" default="false"/>
   <xacro:include filename="$(find net_ft_description)/urdf/net_ft_sensor.xacro"/>
-  <xacro:macro name="ft_sensor_schunk_axia80" params="prefix parent fake_hardware">
-    <!-- TODO: include the fake_hardware param -->
+  <xacro:macro name="ft_sensor_schunk_axia80" params="prefix parent mock_hardware">
     <xacro:net_ft_sensor
       parent="${parent}"
       prefix="${prefix}"
-      use_physical_hardware="$(arg use_physical_hardware)"
+      use_physical_hardware="${mock_hardware == 'false'}"
       ip_address="$(arg ip_address)"
       rdt_sampling_rate="$(arg rdt_sampling_rate)"
