Commit message: Fix OAK-D Pro camera Xacro file

File: aegis_description/urdf/modules/oakd_pro_camera.xacro (robot description, xacro)
@@ -3,5 +3,5 @@
   <xacro:macro name="oakd_pro_camera" params="parent">
     <joint name="cell_to_camera" type="fixed">
-      <origin xyz="-0.055 0.360 2.006" rpy="${pi} 0 0"/>
+      <origin xyz="0.014 0.33 1.972" rpy="${pi / 2} ${pi / 2} 0"/>
       <parent link="${parent}"/>
       <child link="oakd_pro_camera"/>
@@ -9,5 +9,5 @@
     <link name="oakd_pro_camera">
       <visual>
-        <origin xyz="0 0 0" rpy="0 0 0"/>
+        <origin xyz="-0.031 -0.0555 -0.03" rpy="${pi / 2} 0 ${pi / 2}"/>
         <geometry>
           <mesh filename="package://aegis_description/meshes/oakd_pro_camera.dae" scale="1.0 1.0 1.0"/>
@@ -15,5 +15,5 @@
       </visual>
       <collision>
-        <origin xyz="0 0 0" rpy="0 0 0"/>
+        <origin xyz="-0.031 -0.0555 -0.03" rpy="${pi / 2} 0 ${pi / 2}"/>
         <geometry>
           <mesh filename="package://aegis_description/meshes/oakd_pro_camera.dae" scale="1.0 1.0 1.0"/>
