Commit message: ADD: basler lens

File: aegis_description/urdf/modules/basler_camera.xacro (robot description, xacro)
@@ -6,8 +6,9 @@
     <xacro:property name="width" value="0.07002"/>
     <xacro:property name="height" value="0.001353"/>
-    <!-- <xacro:property name="radius2" value="0.0315"/>
-    <xacro:property name="height2" value="0.007"/> -->
     <xacro:property name="camera_mounting_offset" value="0.0387"/>
     <xacro:property name="camera_height" value="0.02900"/>
+    <xacro:property name="lens_radius" value="0.01660"/>
+    <xacro:property name="lens_height" value="0.02890"/>
+    <xacro:property name="lens_offset" value="-0.0145"/>
     <joint name="basler_camera_joint_${side}" type="fixed">
       <origin xyz="0 ${0.5 * camera_height} ${-camera_mounting_offset}" rpy="0 0 0"/>
@@ -21,4 +22,13 @@
           <mesh filename="package://aegis_description/meshes/basler_camera.dae" scale="0.001 0.001 0.001"/>
         </geometry>
+      </visual>
+      <visual>
+        <origin xyz="0 0 ${lens_offset}" rpy="0 0 ${pi}"/>
+        <geometry>
+          <cylinder radius="${lens_radius}" length="${lens_height}"/>
+        </geometry>
+        <material name="black">
+          <color rgba="0.04 0.04 0.04 1"/>
+        </material>
       </visual>
       <!-- <xacro:cylinders_inertial r1="${radius1}" l1="${height1}" r2="${radius2}" l2="${height2}" m="${mass}"/>

Commit message: ADD: camera collision

File: aegis_description/urdf/modules/basler_camera.xacro (robot description, xacro)
@@ -3,9 +3,11 @@
   <!-- <xacro:include filename="$(find aegis_description)/urdf/cylinders_inertial.xacro"/> -->
   <xacro:macro name="basler_camera" params="prefix parent side">
-    <xacro:property name="mass" value="0.217"/>
-    <xacro:property name="width" value="0.07002"/>
-    <xacro:property name="height" value="0.001353"/>
+    <xacro:property name="camera_mass" value="0.217"/>
+    <xacro:property name="lens_mass" value="0.063"/>
+    <!-- <xacro:property name="width" value="0.07002"/>
+    <xacro:property name="height" value="0.001353"/> -->
     <xacro:property name="camera_mounting_offset" value="0.0387"/>
     <xacro:property name="camera_height" value="0.02900"/>
+    <xacro:property name="camera_length" value="0.05400"/>
     <xacro:property name="lens_radius" value="0.01660"/>
     <xacro:property name="lens_height" value="0.02890"/>
@@ -32,17 +34,18 @@
         </material>
       </visual>
-      <!-- <xacro:cylinders_inertial r1="${radius1}" l1="${height1}" r2="${radius2}" l2="${height2}" m="${mass}"/>
+      <!-- <xacro:cylinders_inertial r1="${radius1}" l1="${height1}" r2="${radius2}" l2="${height2}" m="${mass}"/> -->
       <collision>
+        <origin xyz="0 0 0" rpy="0 0 0"/>
         <geometry>
-          <cylinder radius="${radius1}" length="${height1 + height2}"/>
+            <box size="${camera_height} ${camera_height} ${camera_length}" />
         </geometry>
-      </collision> -->
+      </collision>
+      <collision>
+        <origin xyz="0 0 ${lens_offset}" rpy="0 0 ${pi}"/>
+        <geometry>
+          <cylinder radius="${lens_radius}" length="${lens_height}"/>
+        </geometry>
+      </collision>
     </link>
-    <!-- <joint name="${prefix}adapter_from_sensor_end_joint" type="fixed">
-      <origin xyz="0 0 ${height2}" rpy="0 0 0"/>
-      <parent link="${prefix}adapter_from_sensor"/>
-      <child link="${prefix}adapter_from_sensor_end"/>
-    </joint>
-    <link name="${prefix}adapter_from_sensor_end"/> -->
   </xacro:macro>
 </robot>

Commit message: DEL: commented innecessary code

File: aegis_description/urdf/modules/basler_camera.xacro (robot description, xacro)
@@ -5,6 +5,4 @@
     <xacro:property name="camera_mass" value="0.217"/>
     <xacro:property name="lens_mass" value="0.063"/>
-    <!-- <xacro:property name="width" value="0.07002"/>
-    <xacro:property name="height" value="0.001353"/> -->
     <xacro:property name="camera_mounting_offset" value="0.0387"/>
     <xacro:property name="camera_height" value="0.0290"/>

File: aegis_description/urdf/modules/basler_camera_mounting.xacro (robot description, xacro)
@@ -8,11 +8,4 @@
     <xacro:property name="mounting_size_x" value="0.09070"/>
     <xacro:property name="mounting_size_z" value="0.09773"/>
-    <!-- <xacro:property name="mounting_insert_depth" value="0.0076"/> -->
-    <!-- <xacro:property name="radius2" value="0.0315"/>
-    <xacro:property name="height2" value="0.007"/> -->
-    <!-- <xacro:property name="mounting_dist_a" value="0.09070"/>
-    <xacro:property name="mounting_dist_b" value="-0.0460"/>
-    <xacro:property name="mounting_dist_c_x" value="-0.03471"/>
-    <xacro:property name="mounting_dist_c_z" value="-0.04136"/> -->
     <xacro:property name="mounting_yaw" value="-0.6981"/>
     <xacro:property name="mounting_dist_z" value="-0.06607"/>

Commit message: FIX: typos

File: aegis_description/urdf/modules/basler_camera.xacro (robot description, xacro)
@@ -36,5 +36,5 @@
         <origin xyz="0 0 ${0.5 * camera_length}" rpy="0 0 0"/>
         <geometry>
-            <box size="${camera_height} ${camera_height} ${camera_length}"/>
+          <box size="${camera_height} ${camera_height} ${camera_length}"/>
         </geometry>
       </collision>

File: aegis_description/urdf/modules/basler_camera_mounting.xacro (robot description, xacro)
@@ -27,5 +27,5 @@
         <origin xyz="${1.0 * mounting_size_x} 0 ${-1.0 * mounting_height}" rpy="0 0 0"/>
         <geometry>
-          <box size="${mounting_size_x} ${mounting_width} ${3.0 * mounting_height}" />
+          <box size="${mounting_size_x} ${mounting_width} ${3.0 * mounting_height}"/>
         </geometry>
       </collision>

Commit message: DEL: duplicate values in urdf

File: aegis_description/urdf/modules/basler_camera.xacro (robot description, xacro)
@@ -4,10 +4,7 @@
   <xacro:macro name="basler_camera" params="prefix parent side">
     <xacro:property name="camera_mass" value="0.217"/>
-    <xacro:property name="lens_mass" value="0.063"/>
     <xacro:property name="camera_mounting_offset" value="0.0387"/>
     <xacro:property name="camera_height" value="0.0290"/>
     <xacro:property name="camera_length" value="0.0603"/>
-    <xacro:property name="lens_radius" value="0.01660"/>
-    <xacro:property name="lens_height" value="0.02890"/>
     <xacro:property name="lens_offset" value="-0.0145"/>
     <joint name="basler_camera_joint_${side}" type="fixed">

File: aegis_description/urdf/modules/computar_lens.xacro (robot description, xacro)
@@ -3,12 +3,7 @@
   <!-- <xacro:include filename="$(find aegis_description)/urdf/cylinders_inertial.xacro"/> -->
   <xacro:macro name="computar_lens" params="prefix parent side">
-    <xacro:property name="camera_mass" value="0.217"/>
     <xacro:property name="lens_mass" value="0.063"/>
-    <xacro:property name="camera_mounting_offset" value="0.0387"/>
-    <xacro:property name="camera_height" value="0.0290"/>
-    <xacro:property name="camera_length" value="0.0603"/>
     <xacro:property name="lens_radius" value="0.01660"/>
     <xacro:property name="lens_height" value="0.02890"/>
-    <xacro:property name="lens_offset" value="-0.0145"/>
     <joint name="computar_lens_joint_${side}" type="fixed">
       <origin xyz="0 0 0" rpy="0 0 0"/>
