Commit message: Change sensor orientation

File: aegis_description/urdf/modules/ft_schunk_axia80.xacro (robot description, xacro)
@@ -24,5 +24,5 @@
       use_hardware_biasing="$(arg use_hardware_biasing)"
     >
-      <origin xyz="0 0 0" rpy="0 0 0"/>
+      <origin xyz="0 0 0" rpy="0 0 ${pi}"/>
     </xacro:net_ft_sensor>
   </xacro:macro>
