Commit message: Change collision

File: aegis_description/urdf/modules/mount_camera_tool_luxonis.xacro (robot description, xacro)
@@ -18,7 +18,7 @@
       </visual>
       <collision>
-        <origin xyz="0.082 0 -0.028" rpy="0 0 0"/>
+        <origin xyz="0.084 0 -0.01" rpy="0 0 0"/>
         <geometry>
-          <box size="0.082 0.12 0.092"/>
+          <box size="0.076 0.1 0.12"/>
         </geometry>
       </collision>
