Commit message: ADD: origin for camera mountings and measurements of a new adapter

File: aegis_description/urdf/modules/adapter_to_sensor.xacro (robot description, xacro)
@@ -8,4 +8,7 @@
     <xacro:property name="radius2" value="0.04255"/>
     <xacro:property name="height2" value="0.0094"/>
+    <xacro:property name="height_to_adapter" value="0.01456"/>
+    <xacro:property name="height_total" value="0.02080"/>
+    <xacro:property name="width" value="0.08580"/>
     <joint name="${prefix}adapter_to_sensor_joint" type="fixed">
       <origin xyz="0 0 0" rpy="0 0 0"/>
@@ -47,15 +50,15 @@
     <link name="${prefix}adapter_to_sensor_end"/>
     <joint name="${prefix}adapter_to_camera_mounting_back_joint" type="fixed">
-      <origin xyz="0 ${radius2} 0" rpy="0 ${pi} 0"/>
+      <origin xyz="0 0 ${height_to_adapter}" rpy="0 ${pi} 0"/>
       <parent link="${prefix}adapter_to_sensor"/>
       <child link="${prefix}adapter_to_camera_mounting_back"/>
     </joint>
     <link name="${prefix}adapter_to_camera_mounting_back"/>
-    <joint name="${prefix}adapter_to_camera_mounting_front_joint" type="fixed">
+    <!-- <joint name="${prefix}adapter_to_camera_mounting_front_joint" type="fixed">
       <origin xyz="0 ${radius2} 0" rpy="0 ${pi} 0"/>
       <parent link="${prefix}adapter_to_sensor"/>
       <child link="${prefix}adapter_to_camera_mounting_front"/>
     </joint>
-    <link name="${prefix}adapter_to_camera_mounting_front"/>
+    <link name="${prefix}adapter_to_camera_mounting_front"/> -->
   </xacro:macro>
 </robot>

File: aegis_description/urdf/modules/basler_camera_mounting.xacro (robot description, xacro)
@@ -4,10 +4,10 @@
   <xacro:macro name="basler_camera_mounting" params="prefix parent">
     <xacro:property name="mass" value="0.217"/>
-    <xacro:property name="radius1" value="0.041"/>
-    <xacro:property name="height1" value="0.0119"/>
-    <xacro:property name="radius2" value="0.0315"/>
-    <xacro:property name="height2" value="0.007"/>
+    <xacro:property name="mounting_width" value="0.07002"/>
+    <xacro:property name="mounting_height" value="0.001353"/>
+    <!-- <xacro:property name="radius2" value="0.0315"/>
+    <xacro:property name="height2" value="0.007"/> -->
     <joint name="basler_camera_mounting_joint" type="fixed">
-      <origin xyz="0 0 0" rpy="0 0 0"/>
+      <origin xyz="0 0 ${0.5 * mounting_height}" rpy="0 0 0"/>
       <parent link="${parent}"/>
       <child link="${prefix}basler_camera_mounting"/>

Commit message: ADD:  origin to front mounting

File: aegis_description/urdf/modules/adapter_to_sensor.xacro (robot description, xacro)
@@ -26,13 +26,4 @@
         </material>
       </visual>
-      <!-- <visual>
-        <origin xyz="0 0 ${height1 + 0.5 * height2}" rpy="0 0 0"/>
-        <geometry>
-          <cylinder radius="${radius2}" length="${height2}"/>
-        </geometry>
-        <material name="black">
-          <color rgba="0.04 0.04 0.04 1"/>
-        </material>
-      </visual> -->
       <xacro:cylinders_inertial r1="${radius1}" l1="${height1}" r2="${radius2}" l2="${height2}" m="${mass}"/>
       <collision>
@@ -55,10 +46,10 @@
     </joint>
     <link name="${prefix}adapter_to_camera_mounting_back"/>
-    <!-- <joint name="${prefix}adapter_to_camera_mounting_front_joint" type="fixed">
-      <origin xyz="0 ${radius2} 0" rpy="0 ${pi} 0"/>
+    <joint name="${prefix}adapter_to_camera_mounting_front_joint" type="fixed">
+      <origin xyz="0 0 ${height_to_adapter}" rpy="0 ${pi} ${pi}"/>
       <parent link="${prefix}adapter_to_sensor"/>
       <child link="${prefix}adapter_to_camera_mounting_front"/>
     </joint>
-    <link name="${prefix}adapter_to_camera_mounting_front"/> -->
+    <link name="${prefix}adapter_to_camera_mounting_front"/>
   </xacro:macro>
 </robot>

Commit message: ADD: collision to camera mounting

File: aegis_description/urdf/modules/adapter_to_sensor.xacro (robot description, xacro)
@@ -8,6 +8,6 @@
     <xacro:property name="radius2" value="0.04255"/>
     <xacro:property name="height2" value="0.0094"/>
-    <xacro:property name="height_to_adapter" value="0.01456"/>
-    <xacro:property name="height_total" value="0.02080"/>
+    <xacro:property name="height_to_adapter" value="0.0135"/>
+    <xacro:property name="height_total" value="0.0210"/>
     <xacro:property name="width" value="0.0860"/>
     <joint name="${prefix}adapter_to_sensor_joint" type="fixed">
@@ -18,5 +18,5 @@
     <link name="${prefix}adapter_to_sensor">
       <visual>
-        <origin xyz="0 0 0.021" rpy="0 ${pi} ${pi}"/>
+        <origin xyz="0 0 ${height_total}" rpy="0 ${pi} ${pi}"/>
         <geometry>
            <mesh filename="package://aegis_description/meshes/adapter_to_sensor.dae" scale="0.001 0.001 0.001"/>
@@ -28,12 +28,12 @@
       <xacro:cylinders_inertial r1="${radius1}" l1="${height1}" r2="${radius2}" l2="${height2}" m="${mass}"/>
       <collision>
-        <origin xyz="0 0 ${0.5 * (height1 + height2)}" rpy="0 0 0"/>
+        <origin xyz="0 0 ${0.5 * height_total}" rpy="0 0 0"/>
         <geometry>
-          <cylinder radius="${radius2}" length="${height1 + height2}"/>
+          <box size="${width} ${width} ${height_total}" />
         </geometry>
       </collision>
     </link>
     <joint name="${prefix}adapter_to_sensor_end_joint" type="fixed">
-      <origin xyz="0 0 ${height1 + height2}" rpy="0 0 0"/>
+      <origin xyz="0 0 ${height_total}" rpy="0 0 0"/>
       <parent link="${prefix}adapter_to_sensor"/>
       <child link="${prefix}adapter_to_sensor_end"/>

File: aegis_description/urdf/modules/basler_camera.xacro (robot description, xacro)
@@ -8,6 +8,6 @@
     <xacro:property name="height" value="0.001353"/> -->
     <xacro:property name="camera_mounting_offset" value="0.0387"/>
-    <xacro:property name="camera_height" value="0.02900"/>
-    <xacro:property name="camera_length" value="0.05400"/>
+    <xacro:property name="camera_height" value="0.0290"/>
+    <xacro:property name="camera_length" value="0.0603"/>
     <xacro:property name="lens_radius" value="0.01660"/>
     <xacro:property name="lens_height" value="0.02890"/>
@@ -36,5 +36,5 @@
       <!-- <xacro:cylinders_inertial r1="${radius1}" l1="${height1}" r2="${radius2}" l2="${height2}" m="${mass}"/> -->
       <collision>
-        <origin xyz="0 0 0" rpy="0 0 0"/>
+        <origin xyz="0 0 ${0.5 * camera_length}" rpy="0 0 0"/>
         <geometry>
             <box size="${camera_height} ${camera_height} ${camera_length}" />

File: aegis_description/urdf/modules/basler_camera_mounting.xacro (robot description, xacro)
@@ -5,5 +5,7 @@
     <xacro:property name="mass" value="0.217"/>
     <xacro:property name="mounting_width" value="0.07000"/>
-    <xacro:property name="mounting_height" value="0.001353"/>
+    <xacro:property name="mounting_height" value="0.01360"/>
+    <xacro:property name="mounting_size_x" value="0.09070"/>
+    <xacro:property name="mounting_size_z" value="0.09773"/>
     <!-- <xacro:property name="mounting_insert_depth" value="0.0076"/> -->
     <!-- <xacro:property name="radius2" value="0.0315"/>
@@ -17,5 +19,5 @@
     <xacro:property name="mounting_dist_x" value="0.119084"/>
     <joint name="basler_camera_mounting_joint_${side}" type="fixed">
-      <origin xyz="0 0 ${0.5 * mounting_height}" rpy="0 0 0"/>
+      <origin xyz="0 0 0" rpy="0 0 0"/>
       <parent link="${parent}"/>
       <child link="${prefix}basler_camera_mounting_${side}"/>
@@ -28,17 +30,12 @@
         </geometry>
       </visual>
-      <!-- <xacro:cylinders_inertial r1="${radius1}" l1="${height1}" r2="${radius2}" l2="${height2}" m="${mass}"/>
+      <!-- <xacro:cylinders_inertial r1="${radius1}" l1="${height1}" r2="${radius2}" l2="${height2}" m="${mass}"/> -->
       <collision>
+        <origin xyz="${1.0 * mounting_size_x} 0 ${-1.0 * mounting_height}" rpy="0 0 0"/>
         <geometry>
-          <cylinder radius="${radius1}" length="${height1 + height2}"/>
+         <box size="${mounting_size_x} ${mounting_width} ${3.0 * mounting_height}" />
         </geometry>
-      </collision> -->
+      </collision>
     </link>
-    <!-- <joint name="${prefix}adapter_from_sensor_end_joint" type="fixed">
-      <origin xyz="0 0 ${height2}" rpy="0 0 0"/>
-      <parent link="${prefix}adapter_from_sensor"/>
-      <child link="${prefix}adapter_from_sensor_end"/>
-    </joint>
-    <link name="${prefix}adapter_from_sensor_end"/> -->
     <joint name="${prefix}mounting_to_camera_${side}_joint" type="fixed">
       <origin

Commit message: CHG: changelog and precommit issues

File: aegis_description/urdf/modules/adapter_to_sensor.xacro (robot description, xacro)
@@ -20,5 +20,5 @@
         <origin xyz="0 0 ${height_total}" rpy="0 ${pi} ${pi}"/>
         <geometry>
-           <mesh filename="package://aegis_description/meshes/adapter_to_sensor.dae" scale="0.001 0.001 0.001"/>
+          <mesh filename="package://aegis_description/meshes/adapter_to_sensor.dae" scale="0.001 0.001 0.001"/>
         </geometry>
         <material name="black">
@@ -30,5 +30,5 @@
         <origin xyz="0 0 ${0.5 * height_total}" rpy="0 0 0"/>
         <geometry>
-          <box size="${width} ${width} ${height_total}" />
+          <box size="${width} ${width} ${height_total}"/>
         </geometry>
       </collision>

File: aegis_description/urdf/modules/basler_camera.xacro (robot description, xacro)
@@ -36,5 +36,5 @@
         <origin xyz="0 0 ${0.5 * camera_length}" rpy="0 0 0"/>
         <geometry>
-            <box size="${camera_height} ${camera_height} ${camera_length}" />
+            <box size="${camera_height} ${camera_height} ${camera_length}"/>
         </geometry>
       </collision>

File: aegis_description/urdf/modules/basler_camera_mounting.xacro (robot description, xacro)
@@ -27,12 +27,10 @@
         <origin xyz="${1.0 * mounting_size_x} 0 ${-1.0 * mounting_height}" rpy="0 0 0"/>
         <geometry>
-         <box size="${mounting_size_x} ${mounting_width} ${3.0 * mounting_height}" />
+          <box size="${mounting_size_x} ${mounting_width} ${3.0 * mounting_height}" />
         </geometry>
       </collision>
     </link>
     <joint name="${prefix}mounting_to_camera_${side}_joint" type="fixed">
-      <origin
-        xyz="${mounting_dist_x} 0 ${mounting_dist_z}"
-        rpy="${mounting_yaw} 0 ${-0.5 * pi}"/>
+      <origin xyz="${mounting_dist_x} 0 ${mounting_dist_z}" rpy="${mounting_yaw} 0 ${-0.5 * pi}"/>
       <parent link="${prefix}basler_camera_mounting_${side}"/>
       <child link="${prefix}mounting_to_camera_${side}"/>

Commit message: ADD: inertia to new elements

File: aegis_description/urdf/modules/adapter_to_sensor.xacro (robot description, xacro)
@@ -26,5 +26,8 @@
         </material>
       </visual>
-      <xacro:cylinders_inertial r1="${radius1}" l1="${height1}" r2="${radius2}" l2="${height2}" m="${mass}"/>
+      <inertial>
+        <mass value="${mass}"/>
+        <inertia ixx="1e-3" ixy="0.0" ixz="0.0" iyy="1e-3" iyz="0.0" izz="1.9e-3"/>
+      </inertial>
       <collision>
         <origin xyz="0 0 ${0.5 * height_total}" rpy="0 0 0"/>

File: aegis_description/urdf/modules/camera_tool_basler.xacro (robot description, xacro)
@@ -19,5 +19,8 @@
         </geometry>
       </visual>
-      <!-- <xacro:cylinders_inertial r1="${radius1}" l1="${height1}" r2="${radius2}" l2="${height2}" m="${mass}"/> -->
+      <inertial>
+        <mass value="${camera_mass}"/>
+        <inertia ixx="3.403e-1" ixy="2.2385e-5" ixz="1.08974e-2" iyy="3.403e-1" iyz="3.883342" izz="3.9606138e+1"/>
+      </inertial>
       <collision>
         <origin xyz="0 0 ${0.5 * camera_length}" rpy="0 0 0"/>

File: aegis_description/urdf/modules/lens_computar.xacro (robot description, xacro)
@@ -1,5 +1,4 @@
 <?xml version="1.0"?>
 <robot xmlns:xacro="http://ros.org/wiki/xacro">
-  <!-- <xacro:include filename="$(find aegis_description)/urdf/cylinders_inertial.xacro"/> -->
   <xacro:macro name="lens_computar" params="prefix parent side">
     <xacro:property name="lens_mass" value="0.063"/>
@@ -21,4 +20,11 @@
         </material>
       </visual>
+      <inertial>
+        <mass value="${lens_mass}"/>
+        <inertia
+            ixx="${(lens_mass/12.0) * (3*lens_radius*lens_radius + lens_height*lens_height)}"
+            iyy="${(lens_mass/2.0) * (lens_radius*lens_radius)}"
+            izz="${(lens_mass/12.0) * (3*lens_radius*lens_radius + lens_height*lens_height)}"/>
+      </inertial>
       <collision>
         <origin xyz="0 0 0" rpy="0 0 ${pi}"/>

File: aegis_description/urdf/modules/mount_camera_tool_basler.xacro (robot description, xacro)
@@ -22,5 +22,8 @@
         </geometry>
       </visual>
-      <!-- <xacro:cylinders_inertial r1="${radius1}" l1="${height1}" r2="${radius2}" l2="${height2}" m="${mass}"/> -->
+      <inertial>
+        <mass value="${mass}"/>
+        <inertia ixx="1.16e-3" ixy="0.0" ixz="0.37e-3" iyy="1.96e-3" iyz="0.0" izz="1.06e-3"/>
+      </inertial>
       <collision>
         <origin xyz="${1.0 * mounting_size_x} 0 ${-1.0 * mounting_height}" rpy="0 0 0"/>

Commit message: CHG: add origin to inertial

File: aegis_description/urdf/modules/adapter_to_sensor.xacro (robot description, xacro)
@@ -28,4 +28,5 @@
       <inertial>
         <mass value="${mass}"/>
+        <origin xyz="0 0 ${height_total}" rpy="0 ${pi} ${pi}"/>
         <inertia ixx="1e-3" ixy="0.0" ixz="0.0" iyy="1e-3" iyz="0.0" izz="1.9e-3"/>
       </inertial>
