Commit message: Fix inertial parameters

File: aegis_description/urdf/modules/adapter_from_sensor.xacro (robot description, xacro)
@@ -1,17 +1,4 @@
 <?xml version="1.0"?>
 <robot xmlns:xacro="http://ros.org/wiki/xacro">
-  <xacro:macro name="cylinders_inertial" params="r1 l1 r2 l2 m">
-    <inertial>
-      <mass value="${m}"/>
-      <inertia
-        ixx="${0.08333 * m * (3 * (r1 * r1 + r2 * r2) + l1 * l1 + l2 * l2)}"
-        ixy="0.0"
-        ixz="0.0"
-        iyy="${0.08333 * m * (3 * (r1 * r1 + r2 * r2) + l1 * l1 + l2 * l2)}"
-        iyz="0.0"
-        izz="${0.5 * m * (r1 * r1 + r2 * r2)}"
-      />
-    </inertial>
-  </xacro:macro>
   <xacro:macro name="adapter_from_sensor" params="prefix parent">
     <xacro:property name="mass" value="0.217"/>
@@ -32,5 +19,4 @@
         </geometry>
       </visual>
-      <xacro:cylinders_inertial r1="${radius1}" l1="${height1}" r2="${radius2}" l2="${height2}" m="${mass}"/>
       <collision>
         <geometry>
@@ -38,4 +24,9 @@
         </geometry>
       </collision>
+      <inertial>
+        <origin xyz="0 0 0.00839" rpy="0 0 0"/>
+        <mass value="${mass}"/>
+        <inertia ixx="8.740e-5" ixy="0.0" ixz="0.0" iyy="8.740e-5" iyz="0.0" izz="1.631e-4"/>
+      </inertial>
     </link>
     <joint name="${prefix}adapter_from_sensor_end_joint" type="fixed">

File: aegis_description/urdf/modules/adapter_to_sensor.xacro (robot description, xacro)
@@ -25,9 +25,4 @@
         </material>
       </visual>
-      <inertial>
-        <mass value="${mass}"/>
-        <origin xyz="0 0 ${height_total}" rpy="0 ${pi} ${pi}"/>
-        <inertia ixx="1e-3" ixy="0.0" ixz="0.0" iyy="1e-3" iyz="0.0" izz="1.9e-3"/>
-      </inertial>
       <collision>
         <origin xyz="0 0 ${0.5 * height_total}" rpy="0 0 0"/>
@@ -36,4 +31,9 @@
         </geometry>
       </collision>
+      <inertial>
+        <mass value="${mass}"/>
+        <origin xyz="0 0 ${height_total}" rpy="0 ${pi} ${pi}"/>
+        <inertia ixx="1e-3" ixy="0.0" ixz="0.0" iyy="1e-3" iyz="0.0" izz="1.9e-3"/>
+      </inertial>
     </link>
     <joint name="${prefix}adapter_to_sensor_end_joint" type="fixed">

File: aegis_description/urdf/modules/camera_tool_basler.xacro (robot description, xacro)
@@ -2,5 +2,5 @@
 <robot xmlns:xacro="http://ros.org/wiki/xacro">
   <xacro:macro name="camera_tool_basler" params="prefix parent side">
-    <xacro:property name="camera_mass" value="0.217"/>
+    <xacro:property name="camera_mass" value="0.090"/>
     <xacro:property name="camera_mounting_offset" value="-0.0387"/>
     <xacro:property name="camera_height" value="0.0290"/>
@@ -19,8 +19,15 @@
         </geometry>
       </visual>
-      <!-- TODO(issue#46): Fix inertial parameters for tool cameras -->
       <inertial>
+        <origin xyz="0 0 ${0.5 * camera_length}" rpy="0 0 0"/>
         <mass value="${camera_mass}"/>
-        <inertia ixx="0.3403" ixy="0.0" ixz="0.0" iyy="0.3403" iyz="0.0" izz="0.039606138"/>
+        <inertia
+          ixx="${(camera_mass/12.0) * (camera_height*camera_height + camera_length*camera_length)}"
+          ixy="0.0"
+          ixz="0.0"
+          iyy="${(camera_mass/12.0) * (camera_height*camera_height + camera_length*camera_length)}"
+          iyz="0.0"
+          izz="${(camera_mass/6.0) * (camera_height*camera_height)}"
+        />
       </inertial>
     </link>

File: aegis_description/urdf/modules/camera_tool_luxonis.xacro (robot description, xacro)
@@ -20,4 +20,24 @@
       rs_compat="$(arg tool_camera_rs_compat)"
     />
+    <xacro:property name="oak_mass" value="0.300"/>
+    <joint name="${prefix}cam_tool_front_inertia_joint" type="fixed">
+      <origin xyz="0.003 -0.019 -0.039" rpy="0 ${pi / 2} 0"/>
+      <parent link="${parent}"/>
+      <child link="${prefix}cam_tool_front_inertia"/>
+    </joint>
+    <link name="${prefix}cam_tool_front_inertia">
+      <inertial>
+        <origin xyz="0.00005 -0.00298 -0.01266" rpy="0 0 0"/>
+        <mass value="${oak_mass}"/>
+        <inertia
+          ixx="1.140e-4"
+          ixy="0.0"
+          ixz="0.0"
+          iyy="2.018e-4"
+          iyz="0.0"
+          izz="2.165e-4"
+        />
+      </inertial>
+    </link>
   </xacro:macro>
 </robot>

File: aegis_description/urdf/modules/lighting_support_left.xacro (robot description, xacro)
@@ -29,6 +29,6 @@
       </collision>
       <inertial>
+        <origin xyz="0 0 0" rpy="0 0 0"/>
         <mass value="0.1"/>
-        <origin xyz="0 0 0" rpy="0 0 0"/>
         <inertia ixx="0.0001" ixy="0.0" ixz="0.0" iyy="0.0001" iyz="0.0" izz="0.0001"/>
       </inertial>

File: aegis_description/urdf/modules/lighting_support_right.xacro (robot description, xacro)
@@ -23,6 +23,6 @@
       </xacro:unless>
       <inertial>
+        <origin xyz="0 0 0" rpy="0 0 0"/>
         <mass value="0.1"/>
-        <origin xyz="0 0 0" rpy="0 0 0"/>
         <inertia ixx="0.0001" ixy="0.0" ixz="0.0" iyy="0.0001" iyz="0.0" izz="0.0001"/>
       </inertial>

File: aegis_description/urdf/modules/mount_camera_tool_basler.xacro (robot description, xacro)
@@ -2,5 +2,5 @@
 <robot xmlns:xacro="http://ros.org/wiki/xacro">
   <xacro:macro name="mount_camera_tool_basler" params="prefix parent side">
-    <xacro:property name="mass" value="0.217"/>
+    <xacro:property name="mass" value="0.054"/>
     <xacro:property name="mounting_width" value="0.07000"/>
     <xacro:property name="mounting_height" value="0.01360"/>
@@ -22,9 +22,4 @@
         </geometry>
       </visual>
-      <!-- TODO(issue#46): Fix inertial parameters for tool cameras -->
-      <inertial>
-        <mass value="${mass}"/>
-        <inertia ixx="116e-6" ixy="0" ixz="37.5e-6" iyy="196e-6" iyz="0" izz="106e-6"/>
-      </inertial>
       <collision>
         <origin xyz="0.048 0 0" rpy="0 0 0"/>
@@ -57,4 +52,16 @@
         </geometry>
       </collision>
+      <inertial>
+        <origin xyz="0.09912 0 -0.02301" rpy="0 0 0"/>
+        <mass value="${mass}"/>
+        <inertia
+          ixx="5.227e-5"
+          ixy="0.0"
+          ixz="1.688e-5"
+          iyy="8.825e-5"
+          iyz="0.0"
+          izz="4.786e-5"
+        />
+      </inertial>
     </link>
     <joint name="${prefix}mount_${side}_end_joint" type="fixed">

File: aegis_description/urdf/modules/mount_camera_tool_luxonis.xacro (robot description, xacro)
@@ -2,5 +2,5 @@
 <robot xmlns:xacro="http://ros.org/wiki/xacro">
   <xacro:macro name="mount_camera_tool_luxonis" params="prefix parent">
-    <xacro:property name="mass" value="0.4"/>
+    <xacro:property name="mass" value="0.026"/>
     <joint name="${prefix}mount_front_joint" type="fixed">
       <origin xyz="0 0 0" rpy="0 0 0"/>
@@ -15,9 +15,4 @@
         </geometry>
       </visual>
-      <!-- TODO(issue#46): Fix inertial parameters for tool cameras -->
-      <inertial>
-        <mass value="${mass}"/>
-        <inertia ixx="27.3e-6" ixy="0" ixz="4.19e-6" iyy="19.7e-6" iyz="0" izz="43.38e-6"/>
-      </inertial>
       <collision>
         <origin xyz="0.084 0 0" rpy="0 0 0"/>
@@ -26,4 +21,16 @@
         </geometry>
       </collision>
+      <inertial>
+        <origin xyz="0.06944 0 -0.00584" rpy="0 0 0"/>
+        <mass value="${mass}"/>
+        <inertia
+          ixx="1.318e-5"
+          ixy="0.0"
+          ixz="2.022e-6"
+          iyy="9.518e-6"
+          iyz="0.0"
+          izz="2.094e-5"
+        />
+      </inertial>
     </link>
     <joint name="${prefix}mount_front_end_joint" type="fixed">

Commit message: Moved 90 deg gripper rotation to FT package

File: aegis_description/urdf/modules/adapter_from_sensor.xacro (robot description, xacro)
@@ -31,5 +31,5 @@
     </link>
     <joint name="${prefix}adapter_from_sensor_end_joint" type="fixed">
-      <origin xyz="0 0 ${height2}" rpy="0 0 ${0.5 * pi}"/>
+      <origin xyz="0 0 ${height2}" rpy="0 0 0"/>
       <parent link="${prefix}adapter_from_sensor"/>
       <child link="${prefix}adapter_from_sensor_end"/>
