Commit message: CHG: mount and camera mesh files names

File: aegis_description/urdf/modules/camera_tool_basler.xacro (robot description, xacro)
@@ -16,5 +16,5 @@
         <origin xyz="0 0 0" rpy="0 0 0"/>
         <geometry>
-          <mesh filename="package://aegis_description/meshes/basler_camera.dae" scale="0.001 0.001 0.001"/>
+          <mesh filename="package://aegis_description/meshes/camera_tool_basler.dae" scale="0.001 0.001 0.001"/>
         </geometry>
       </visual>

File: aegis_description/urdf/modules/mount_camera_tool_basler.xacro (robot description, xacro)
@@ -19,5 +19,5 @@
         <origin xyz="0 0 0" rpy="0 0 0"/>
         <geometry>
-          <mesh filename="package://aegis_description/meshes/basler_camera_mounting.dae" scale="0.001 0.001 0.001"/>
+          <mesh filename="package://aegis_description/meshes/mount_camera_tool_basler.dae" scale="0.001 0.001 0.001"/>
         </geometry>
       </visual>

Commit message: FIX: camera tool basler inertia

File: aegis_description/urdf/modules/camera_tool_basler.xacro (robot description, xacro)
@@ -21,5 +21,5 @@
       <inertial>
         <mass value="${camera_mass}"/>
-        <inertia ixx="3.403e-1" ixy="2.2385e-5" ixz="1.08974e-2" iyy="3.403e-1" iyz="3.883342" izz="3.9606138e+1"/>
+        <inertia ixx="0.3403" ixy="0.0" ixz="0.0" iyy="0.3403" iyz="0.0" izz="0.039606138"/>
       </inertial>
       <collision>

Commit message: CHG: pr comments

File: aegis_description/urdf/modules/camera_tool_basler.xacro (robot description, xacro)
@@ -3,10 +3,10 @@
   <xacro:macro name="camera_tool_basler" params="prefix parent side">
     <xacro:property name="camera_mass" value="0.217"/>
-    <xacro:property name="camera_mounting_offset" value="0.0387"/>
+    <xacro:property name="camera_mounting_offset" value="-0.0387"/>
     <xacro:property name="camera_height" value="0.0290"/>
     <xacro:property name="camera_length" value="0.0603"/>
     <xacro:property name="lens_offset" value="-0.0145"/>
     <joint name="basler_camera_joint_${side}" type="fixed">
-      <origin xyz="0 ${0.5 * camera_height} ${-camera_mounting_offset}" rpy="0 0 0"/>
+      <origin xyz="0 ${0.5 * camera_height} ${camera_mounting_offset}" rpy="0 0 0"/>
       <parent link="${parent}"/>
       <child link="${prefix}basler_camera_${side}"/>

Commit message: Add TODO comments

File: aegis_description/urdf/modules/camera_tool_basler.xacro (robot description, xacro)
@@ -19,4 +19,5 @@
         </geometry>
       </visual>
+      <!-- TODO(issue#46): Fix inertial parameters for tool cameras -->
       <inertial>
         <mass value="${camera_mass}"/>

File: aegis_description/urdf/modules/mount_camera_tool_basler.xacro (robot description, xacro)
@@ -22,7 +22,8 @@
         </geometry>
       </visual>
+      <!-- TODO(issue#46): Fix inertial parameters for tool cameras -->
       <inertial>
         <mass value="${mass}"/>
-        <inertia ixx="1.16e-3" ixy="0.0" ixz="0.37e-3" iyy="1.96e-3" iyz="0.0" izz="1.06e-3"/>
+        <inertia ixx="116e-6" ixy="0" ixz="37.5e-6" iyy="196e-6" iyz="0" izz="106e-6"/>
       </inertial>
       <collision>

File: aegis_description/urdf/modules/mount_camera_tool_luxonis.xacro (robot description, xacro)
@@ -17,4 +17,9 @@
         </geometry>
       </visual>
+      <!-- TODO(issue#46): Fix inertial parameters for tool cameras -->
+      <inertial>
+        <mass value="${mass}"/>
+        <inertia ixx="27.3e-6" ixy="0" ixz="4.19e-6" iyy="19.7e-6" iyz="0" izz="43.38e-6"/>
+      </inertial>
       <collision>
         <origin xyz="0.084 0 -0.01" rpy="0 0 0"/>
