Commit message: win on robot description

File: aegis_description/urdf/modules/ur_definition.xacro (robot description, xacro)
@@ -2,5 +2,5 @@
 <robot xmlns:xacro="http://ros.org/wiki/xacro">
   <xacro:include filename="$(find ur_description)/urdf/ur_macro.xacro"/>
-  <xacro:macro name="ur_definition" params="name parent prefix kinematics_calibration fake_hardware">
+  <xacro:macro name="ur_definition" params="name parent prefix kinematics_calibration mock_hardware">
     <!-- possible 'ur_type' values: ur3, ur3e, ur5, ur5e, ur10, ur10e, ur16e, ur20 -->
     <!-- the default value should raise an error in case this was called without defining the
@@ -39,5 +39,5 @@
     <xacro:arg name="tool_tcp_port" default="54321"/>
     <!-- Simulation parameters -->
-    <xacro:arg name="use_fake_hardware" default="${fake_hardware}"/>
+    <xacro:arg name="use_fake_hardware" default="${mock_hardware}"/>
     <xacro:arg name="fake_sensor_commands" default="false"/>
     <xacro:arg name="sim_gazebo" default="false"/>
@@ -45,6 +45,5 @@
     <xacro:arg name="simulation_controllers" default=""/>
     <!-- initial position for simulations (Fake Hardware, Gazebo, Ignition) -->
-    <!-- TODO: remap this to our aegis_control package -->
-    <xacro:arg name="initial_positions_file" default="$(find ur_description)/config/initial_positions.yaml"/>
+    <xacro:arg name="initial_positions_file" default="$(find aegis_control)/config/initial_positions.yaml"/>
     <!-- convert to property to use substitution in function -->
     <xacro:property name="initial_positions_file" default="$(arg initial_positions_file)"/>
@@ -58,32 +57,4 @@
       physical_parameters_file="$(arg physical_params)"
       visual_parameters_file="$(arg visual_params)"
-      transmission_hw_interface="$(arg transmission_hw_interface)"
-      safety_limits="$(arg safety_limits)"
-      safety_pos_margin="$(arg safety_pos_margin)"
-      safety_k_position="$(arg safety_k_position)"
-      use_fake_hardware="$(arg use_fake_hardware)"
-      fake_sensor_commands="$(arg fake_sensor_commands)"
-      sim_gazebo="$(arg sim_gazebo)"
-      sim_ignition="$(arg sim_ignition)"
-      headless_mode="$(arg headless_mode)"
-      initial_positions="${xacro.load_yaml(initial_positions_file)}"
-      use_tool_communication="$(arg use_tool_communication)"
-      tool_voltage="$(arg tool_voltage)"
-      tool_parity="$(arg tool_parity)"
-      tool_baud_rate="$(arg tool_baud_rate)"
-      tool_stop_bits="$(arg tool_stop_bits)"
-      tool_rx_idle_chars="$(arg tool_rx_idle_chars)"
-      tool_tx_idle_chars="$(arg tool_tx_idle_chars)"
-      tool_device_name="$(arg tool_device_name)"
-      tool_tcp_port="$(arg tool_tcp_port)"
-      robot_ip="$(arg robot_ip)"
-      script_filename="$(arg script_filename)"
-      output_recipe_filename="$(arg output_recipe_filename)"
-      input_recipe_filename="$(arg input_recipe_filename)"
-      reverse_ip="$(arg reverse_ip)"
-      script_command_port="$(arg script_command_port)"
-      reverse_port="$(arg reverse_port)"
-      script_sender_port="$(arg script_sender_port)"
-      trajectory_port="$(arg trajectory_port)"
     >
       <!-- position robot in the world -->

Commit message: CHG: fixes around world-ur_base reference

File: aegis_description/urdf/modules/ur_definition.xacro (robot description, xacro)
@@ -2,13 +2,13 @@
 <robot xmlns:xacro="http://ros.org/wiki/xacro">
   <xacro:include filename="$(find ur_description)/urdf/ur_macro.xacro"/>
-  <!-- For simulation, the global parent must be the same as ur_base -->
-  <joint name="world_to_ur_base" type="fixed">
-    <origin xyz="0 0 0" rpy="0 0 0"/>
-    <parent link="${parent}"/>
-    <child link="ur_base"/>
-  </joint>
   <!-- The list of all available options can be found in the <ur_description>/urdf/ur_macro.xacro file -->
   <!-- Descriptions of the arguments can be found in the <ur_robot_driver>/src/hardware_interface.cpp file -->
   <xacro:macro name="ur_definition" params="name parent tf_prefix mock_hardware">
+    <!-- For simulation, the global parent must be the same as ur_base -->
+    <joint name="world_to_ur_base" type="fixed">
+      <origin xyz="0 0 0" rpy="0 0 0"/>
+      <parent link="${parent}"/>
+      <child link="ur_base"/>
+    </joint>
     <!-- parameters -->
     <xacro:arg name="tf_prefix" default="${tf_prefix}"/>
