Commit message: Change cell collision

File: aegis_description/urdf/modules/cell.xacro (robot description, xacro)
@@ -15,7 +15,31 @@
       </visual>
       <collision>
-        <origin xyz="-0.460 -0.240 0.786" rpy="0 0 0"/>
+        <origin xyz="0 0.06 0.43" rpy="0 0 0"/>
         <geometry>
-          <mesh filename="package://aegis_description/meshes/cell.dae" scale="1.0 1.0 1.0"/>
+          <box size="0.84 0.56 0.86"/>
+        </geometry>
+      </collision>
+      <collision>
+        <origin xyz="-0.48 0 0.96" rpy="0 0 0"/>
+        <geometry>
+          <box size="0.12 0.68 1.92"/>
+        </geometry>
+      </collision>
+      <collision>
+        <origin xyz="0.48 0 0.96" rpy="0 0 0"/>
+        <geometry>
+          <box size="0.12 0.68 1.92"/>
+        </geometry>
+      </collision>
+      <collision>
+        <origin xyz="0 -0.28 0.96" rpy="0 0 0"/>
+        <geometry>
+          <box size="0.84 0.12 1.92"/>
+        </geometry>
+      </collision>
+      <collision>
+        <origin xyz="0 0.04 1.98" rpy="0 0 0"/>
+        <geometry>
+          <box size="1.08 0.76 0.12"/>
         </geometry>
       </collision>

Commit message: Change cell collision

File: aegis_description/urdf/modules/cell.xacro (robot description, xacro)
@@ -15,31 +15,37 @@
       </visual>
       <collision>
-        <origin xyz="0 0.06 0.43" rpy="0 0 0"/>
+        <origin xyz="0 0 0.41" rpy="0 0 0"/>
         <geometry>
-          <box size="0.84 0.56 0.86"/>
+          <box size="0.88 0.648 0.82"/>
         </geometry>
       </collision>
       <collision>
-        <origin xyz="-0.48 0 0.96" rpy="0 0 0"/>
+        <origin xyz="0.48 0 0.97" rpy="0 0 0"/>
         <geometry>
-          <box size="0.12 0.68 1.92"/>
+          <box size="0.08 0.648 1.94"/>
         </geometry>
       </collision>
       <collision>
-        <origin xyz="0.48 0 0.96" rpy="0 0 0"/>
+        <origin xyz="0.41 0 0.85" rpy="0 0 0"/>
         <geometry>
-          <box size="0.12 0.68 1.92"/>
+          <box size="0.06 0.648 0.06"/>
         </geometry>
       </collision>
       <collision>
-        <origin xyz="0 -0.28 0.96" rpy="0 0 0"/>
+        <origin xyz="-0.48 0 0.97" rpy="0 0 0"/>
         <geometry>
-          <box size="0.84 0.12 1.92"/>
+          <box size="0.08 0.648 1.94"/>
         </geometry>
       </collision>
       <collision>
-        <origin xyz="0 0.04 1.98" rpy="0 0 0"/>
+        <origin xyz="-0.41 0 0.85" rpy="0 0 0"/>
         <geometry>
-          <box size="1.08 0.76 0.12"/>
+          <box size="0.06 0.648 0.06"/>
+        </geometry>
+      </collision>
+      <collision>
+        <origin xyz="0 0.02 1.98" rpy="0 0 0"/>
+        <geometry>
+          <box size="1.04 0.688 0.08"/>
         </geometry>
       </collision>

Commit message: Change cell collision

File: aegis_description/urdf/modules/cell.xacro (robot description, xacro)
@@ -45,7 +45,7 @@
       </collision>
       <collision>
-        <origin xyz="0 0.02 1.98" rpy="0 0 0"/>
+        <origin xyz="0 0.04 1.98" rpy="0 0 0"/>
         <geometry>
-          <box size="1.04 0.688 0.08"/>
+          <box size="1.04 0.728 0.08"/>
         </geometry>
       </collision>

Commit message: Change cell collision

File: aegis_description/urdf/modules/cell.xacro (robot description, xacro)
@@ -15,7 +15,13 @@
       </visual>
       <collision>
-        <origin xyz="0 0 0.41" rpy="0 0 0"/>
+        <origin xyz="0 -0.162 0.435" rpy="0 0 0"/>
         <geometry>
-          <box size="0.88 0.648 0.82"/>
+          <box size="0.72 0.324 0.87"/>
+        </geometry>
+      </collision>
+      <collision>
+        <origin xyz="0 0.162 0.41" rpy="0 0 0"/>
+        <geometry>
+          <box size="0.72 0.324 0.82"/>
         </geometry>
       </collision>
@@ -27,7 +33,7 @@
       </collision>
       <collision>
-        <origin xyz="0.41 0 0.85" rpy="0 0 0"/>
+        <origin xyz="0.4 0 0.435" rpy="0 0 0"/>
         <geometry>
-          <box size="0.06 0.648 0.06"/>
+          <box size="0.08 0.648 0.87"/>
         </geometry>
       </collision>
@@ -39,7 +45,7 @@
       </collision>
       <collision>
-        <origin xyz="-0.41 0 0.85" rpy="0 0 0"/>
+        <origin xyz="-0.4 0 0.435" rpy="0 0 0"/>
         <geometry>
-          <box size="0.06 0.648 0.06"/>
+          <box size="0.08 0.648 0.87"/>
         </geometry>
       </collision>
@@ -48,4 +54,10 @@
         <geometry>
           <box size="1.04 0.728 0.08"/>
+        </geometry>
+      </collision>
+      <collision>
+        <origin xyz="0 -0.62 1.2" rpy="0 0 0"/>
+        <geometry>
+          <box size="2.4 0.02 2.4"/>
         </geometry>
       </collision>

Commit message: Apply suggestions from code review
Co-authored-by: Jakub Plachno <sivral@proton.me>

File: aegis_description/urdf/modules/cell.xacro (robot description, xacro)
@@ -2,5 +2,5 @@
 <robot xmlns:xacro="http://ros.org/wiki/xacro">
   <xacro:macro name="cell" params="parent">
-    <joint name="parent_to_cell" type="fixed">
+    <joint name="world_to_cell" type="fixed">
       <origin xyz="0 0 -0.806" rpy="0 0 -${0.5 * pi}"/>
       <parent link="${parent}"/>

Commit message: Modify cell Xacro file

File: aegis_description/urdf/modules/cell.xacro (robot description, xacro)
@@ -4,5 +4,5 @@
     <xacro:unless value="${disable_cell}">
       <joint name="world_to_cell" type="fixed">
-        <origin xyz="0 0 -0.806" rpy="0 0 -${0.5 * pi}"/>
+        <origin xyz="0 0 -0.821" rpy="0 0 -${0.5 * pi}"/>
         <parent link="${parent}"/>
         <child link="cell"/>
