Commit message: disable_leds argument missing again

File: aegis_description/urdf/modules/cell.xacro (robot description, xacro)
@@ -1,5 +1,5 @@
 <?xml version="1.0"?>
 <robot xmlns:xacro="http://ros.org/wiki/xacro">
-  <xacro:macro name="cell" params="parent disable_cell disable_cell_collision">
+  <xacro:macro name="cell" params="parent disable_cell disable_cell_collision disable_leds">
     <xacro:unless value="${disable_cell}">
       <joint name="world_to_cell" type="fixed">
@@ -66,6 +66,8 @@
         </xacro:unless>
       </link>
-      <xacro:wled_lights_right parent="cell" prefix=""/>
-      <xacro:wled_lights_left parent="cell" prefix=""/>
+      <xacro:unless value="${disable_leds}">
+        <xacro:lighting_support_right parent="cell" prefix=""/>
+        <xacro:lighting_support_left parent="cell" prefix=""/>
+      </xacro:unless>
     </xacro:unless>
   </xacro:macro>

Commit message: aegis_description: Simplified collision mesh of the lightning supports

File: aegis_description/urdf/modules/cell.xacro (robot description, xacro)
@@ -67,6 +67,6 @@
       </link>
       <xacro:unless value="${disable_leds}">
-        <xacro:lighting_support_right parent="cell" prefix=""/>
-        <xacro:lighting_support_left parent="cell" prefix=""/>
+      <xacro:lighting_support_right parent="cell" prefix="" disable_cell_collision="${disable_cell_collision}"/>
+      <xacro:lighting_support_left parent="cell" prefix="" disable_cell_collision="${disable_cell_collision}"/>
       </xacro:unless>
     </xacro:unless>

File: aegis_description/urdf/modules/lighting_support_left.xacro (robot description, xacro)
@@ -1,5 +1,5 @@
 <?xml version="1.0"?>
 <robot xmlns:xacro="http://ros.org/wiki/xacro">
-  <xacro:macro name="lighting_support_left" params="parent prefix">
+  <xacro:macro name="lighting_support_left" params="parent prefix disable_cell_collision">
     <joint name="${prefix}lighting_support_left_joint" type="fixed">
       <origin xyz="0.50 0.30 1.171" rpy="0.0 0.0 ${-0.5 * pi}"/>
@@ -14,4 +14,12 @@
         </geometry>
       </visual>
+      <xacro:unless value="${disable_cell_collision}">
+        <collision>
+          <origin xyz="-0.277 0.007 -0.015" rpy="0 0 0"/>
+          <geometry>
+            <box size="0.6 0.07 0.16"/>
+          </geometry>
+        </collision>
+      </xacro:unless>
       <collision>
         <origin xyz="0 0 0" rpy="0 0 0"/>

File: aegis_description/urdf/modules/lighting_support_right.xacro (robot description, xacro)
@@ -1,5 +1,5 @@
 <?xml version="1.0"?>
 <robot xmlns:xacro="http://ros.org/wiki/xacro">
-  <xacro:macro name="lighting_support_right" params="parent prefix">
+  <xacro:macro name="lighting_support_right" params="parent prefix disable_cell_collision">
     <joint name="${prefix}lighting_support_right_joint" type="fixed">
       <origin xyz="-0.50 0.30 1.171" rpy="0.0 0.0 ${-0.5 * pi}"/>
@@ -14,10 +14,12 @@
         </geometry>
       </visual>
-      <collision>
-        <origin xyz="0 0 0" rpy="0 0 0"/>
-        <geometry>
-          <mesh filename="package://aegis_description/meshes/lighting_support_right.dae" scale="0.001 0.001 0.001"/>
-        </geometry>
-      </collision>
+      <xacro:unless value="${disable_cell_collision}">
+        <collision>
+          <origin xyz="-0.277 -0.007 -0.015" rpy="0 0 0"/>
+          <geometry>
+            <box size="0.6 0.07 0.16"/>
+          </geometry>
+        </collision>
+      </xacro:unless>
       <inertial>
         <mass value="0.1"/>
