Commit message: Update changelog

File: aegis_description/urdf/modules/camera_tool_luxonis.xacro (robot description, xacro)
@@ -30,12 +30,5 @@
         <origin xyz="0.00005 -0.00298 -0.01266" rpy="0 0 0"/>
         <mass value="${oak_mass}"/>
-        <inertia
-          ixx="1.140e-4"
-          ixy="0.0"
-          ixz="0.0"
-          iyy="2.018e-4"
-          iyz="0.0"
-          izz="2.165e-4"
-        />
+        <inertia ixx="1.140e-4" ixy="0.0" ixz="0.0" iyy="2.018e-4" iyz="0.0" izz="2.165e-4"/>
       </inertial>
     </link>

File: aegis_description/urdf/modules/mount_camera_tool_basler.xacro (robot description, xacro)
@@ -55,12 +55,5 @@
         <origin xyz="0.09912 0 -0.02301" rpy="0 0 0"/>
         <mass value="${mass}"/>
-        <inertia
-          ixx="5.227e-5"
-          ixy="0.0"
-          ixz="1.688e-5"
-          iyy="8.825e-5"
-          iyz="0.0"
-          izz="4.786e-5"
-        />
+        <inertia ixx="5.227e-5" ixy="0.0" ixz="1.688e-5" iyy="8.825e-5" iyz="0.0" izz="4.786e-5"/>
       </inertial>
     </link>

File: aegis_description/urdf/modules/mount_camera_tool_luxonis.xacro (robot description, xacro)
@@ -24,12 +24,5 @@
         <origin xyz="0.06944 0 -0.00584" rpy="0 0 0"/>
         <mass value="${mass}"/>
-        <inertia
-          ixx="1.318e-5"
-          ixy="0.0"
-          ixz="2.022e-6"
-          iyy="9.518e-6"
-          iyz="0.0"
-          izz="2.094e-5"
-        />
+        <inertia ixx="1.318e-5" ixy="0.0" ixz="2.022e-6" iyy="9.518e-6" iyz="0.0" izz="2.094e-5"/>
       </inertial>
     </link>
