Commit message: aegis_description: Fixed the obj center of lighting supports

File: aegis_description/urdf/modules/lighting_support_left.xacro (robot description, xacro)
@@ -3,5 +3,5 @@
   <xacro:macro name="lighting_support_left" params="parent prefix">
     <joint name="${prefix}lighting_support_left_joint" type="fixed">
-      <origin xyz="0.32 0.495 0.35" rpy="0.0 0.0 ${pi}"/>
+      <origin xyz="0.50 0.30 1.171" rpy="0.0 0.0 ${-0.5 * pi}"/>
       <parent link="${parent}"/>
       <child link="${prefix}lighting_support_left_link"/>

File: aegis_description/urdf/modules/lighting_support_right.xacro (robot description, xacro)
@@ -3,5 +3,5 @@
   <xacro:macro name="lighting_support_right" params="parent prefix">
     <joint name="${prefix}lighting_support_right_joint" type="fixed">
-      <origin xyz="0.32 0.50 0.35" rpy="0.0 0.0 ${pi}"/>
+      <origin xyz="-0.50 0.30 1.171" rpy="0.0 0.0 ${-0.5 * pi}"/>
       <parent link="${parent}"/>
       <child link="${prefix}lighting_support_right_link"/>

Commit message: Fixed double definition of the collision

File: aegis_description/urdf/modules/lighting_support_left.xacro (robot description, xacro)
@@ -22,10 +22,4 @@
         </collision>
       </xacro:unless>
-      <collision>
-        <origin xyz="0 0 0" rpy="0 0 0"/>
-        <geometry>
-          <mesh filename="package://aegis_description/meshes/lighting_support_left.dae" scale="0.001 0.001 0.001"/>
-        </geometry>
-      </collision>
       <inertial>
         <origin xyz="0 0 0" rpy="0 0 0"/>
